File: BMS1/BMS1.kicad_sch (KiCad schematic)
At the start: 70 parts, among them J1 Conn_01x02, J2 Conn_01x02, J3 Conn_01x02, Q1 Q_NPN_BCE, Q2 Q_NPN_BCE, T1 ESMIT-4180_C, U1 ADG728, U10 LTC6812-1, U2 ADG728, U3 ADG728, U4 ADG728, U5 ADG728, U6 ADG728, U7 ADG728, U8 ADG728, U9 LTC6812-1

Commit message: Everybody is in their general local!
Connections:
- net GND1: now also C14.2
- net GND2: now also C13.2
- removed net GND: C13.2, C14.2
Changed lines of the file:
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@@
-    )
-  )
-  (symbol (lib_id "power:GND") (at 83.185 30.607 0) (unit 1)
-    (in_bom yes) (on_board yes) (dnp no) (fields_autoplaced)
-    (property "Reference" "#PWR061" (at 83.185 36.957 0)
-      (effects (font (size 1.27 1.27)) hide)
-    )
-    (property "Value" "GND" (at 83.185 35.433 0)
-      (effects (font (size 1.27 1.27)))
-    )
-    (property "Footprint" "" (at 83.185 30.607 0)
-      (effects (font (size 1.27 1.27)) hide)
-    )
-    (property "Datasheet" "" (at 83.185 30.607 0)
-      (effects (font (size 1.27 1.27)) hide)
-    )
-    (pin "1")
-    (instances
-      (project "BMS1"
-        (path "/03933f33-7fdb-43de-9d7d-a565cad8a277"
-          (reference "#PWR061") (unit 1)
-        )
-      )
     )
   )
@@
         (path "/03933f33-7fdb-43de-9d7d-a565cad8a277"
           (reference "#PWR016") (unit 1)
+        )
+      )
+    )
+  )
+  (symbol (lib_id "power:GND1") (at 100.209 151.13 0) (unit 1)
+    (in_bom yes) (on_board yes) (dnp no) (fields_autoplaced)
+    (property "Reference" "#PWR063" (at 100.209 157.48 0)
+      (effects (font (size 1.27 1.27)) hide)
+    )
+    (property "Value" "GND1" (at 100.209 155.829 0)
+      (effects (font (size 1.27 1.27)))
+    )
+    (property "Footprint" "" (at 100.209 151.13 0)
+      (effects (font (size 1.27 1.27)) hide)
+    )
+    (property "Datasheet" "" (at 100.209 151.13 0)
+      (effects (font (size 1.27 1.27)) hide)
+    )
+    (pin "1")
+    (instances
+      (project "BMS1"
+        (path "/03933f33-7fdb-43de-9d7d-a565cad8a277"
+          (reference "#PWR063") (unit 1)
         )
       )
@@
     )
   )
-  (symbol (lib_id "power:GND") (at 100.209 151.13 0) (unit 1)
-    (in_bom yes) (on_board yes) (dnp no) (fields_autoplaced)
-    (property "Reference" "#PWR062" (at 100.209 157.48 0)
-      (effects (font (size 1.27 1.27)) hide)
-    )
-    (property "Value" "GND" (at 100.209 155.956 0)
-      (effects (font (size 1.27 1.27)))
-    )
-    (property "Footprint" "" (at 100.209 151.13 0)
-      (effects (font (size 1.27 1.27)) hide)
-    )
-    (property "Datasheet" "" (at 100.209 151.13 0)
-      (effects (font (size 1.27 1.27)) hide)
-    )
-    (pin "1")
-    (instances
-      (project "BMS1"
-        (path "/03933f33-7fdb-43de-9d7d-a565cad8a277"
-          (reference "#PWR062") (unit 1)
-        )
-      )
-    )
-  )
   (symbol (lib_id "power:GND2") (at 248.666 130.048 0) (unit 1)
     (in_bom yes) (on_board yes) (dnp no) (fields_autoplaced)
@@
         )
       )
+    )
+  )
+  (symbol (lib_id "power:GND2") (at 83.185 30.607 0) (unit 1)
+    (in_bom yes) (on_board yes) (dnp no) (fields_autoplaced)
+    (property "Reference" "#PWR062" (at 83.185 36.957 0)
+      (effects (font (size 1.27 1.27)) hide)
+    )
+    (property "Value" "GND2" (at 83.185 35.179 0)
+      (effects (font (size 1.27 1.27)))
+    )
+    (property "Footprint" "" (at 83.185 30.607 0)
+      (effects (font (size 1.27 1.27)) hide)
+    )
+    (property "Datasheet" "" (at 83.185 30.607 0)
+      (effects (font (size 1.27 1.27)) hide)
+    )
+    (pin "1")
+    (instances
+      (project "BMS1"
+        (path "/03933f33-7fdb-43de-9d7d-a565cad8a277"
+          (reference "#PWR062") (unit 1)
+        )
+      )

Commit message: V1 Layout!
Parts:
- added D1, D2: LED, LED_SMD:LED_0603_1608Metric_Pad1.05x0.95mm_HandSolder, symbol Device:LED
- added R94, R95: R_US, Resistor_SMD:R_0603_1608Metric_Pad0.98x0.95mm_HandSolder, symbol Device:R_US
Connections:
- net GND1: now also R94.1
- net GND2: now also R95.1
- net VD: now also D1.2 (A)
- net VDD: now also D2.2 (A)
- new net: D1.1 (K), R94.2
- new net: D2.1 (K), R95.2

Commit message: Schematic (Self) Review Done
Parts:
- C1, C2, C3, C4, C5, C6, C7, C8: value 100nF -> 15u
Other:
- note added: "Isolation to Car"
- moved on the sheet: J1, T1
Changed lines of the file:
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@@
     (stroke (width 0) (type default))
   )
-  (wire (pts (xy 29.597 222.504) (xy 26.041 222.504))
+  (wire (pts (xy 25.146 223.266) (xy 21.59 223.266))
     (stroke (width 0) (type default))
   )
@@
     (stroke (width 0) (type default))
   )
-  (wire (pts (xy 79.629 43.053) (xy 107.569 43.053))
-    (stroke (width 0) (type default))
-  )
   (wire (pts (xy 266.319 97.028) (xy 266.319 99.568))
     (stroke (width 0) (type default))
@@
     (stroke (width 0) (type default))
   )
+  (wire (pts (xy 79.629 43.053) (xy 107.569 43.053))
+    (stroke (width 0) (type default))
+  )
   (polyline (pts (xy 302.006 136.271) (xy 219.202 136.271))
     (stroke (width 0) (type default))
@@
     (stroke (width 0) (type default))
   )
-  (wire (pts (xy 26.041 222.504) (xy 26.041 229.108))
+  (wire (pts (xy 21.59 223.266) (xy 21.59 229.87))
     (stroke (width 0) (type default))
   )
@@
     (stroke (width 0) (type default))
   )
+  (wire (pts (xy 79.629 37.973) (xy 107.569 37.973))
+    (stroke (width 0) (type default))
+  )
   (polyline (pts (xy 219.202 136.271) (xy 219.202 20.701))
     (stroke (width 0) (type default))
@@
     (stroke (width 0) (type default))
   )
-  (wire (pts (xy 43.821 236.728) (xy 43.821 249.301))
+  (wire (pts (xy 39.37 237.49) (xy 39.37 250.063))
     (stroke (width 0) (type default))
   )
@@
     (stroke (width 0) (type default))
   )
-  (wire (pts (xy 33.534 252.73) (xy 33.534 249.301))
+  (wire (pts (xy 29.083 253.492) (xy 29.083 250.063))
     (stroke (width 0) (type default))
   )
@@
     (stroke (width 0) (type default))
   )
-  (wire (pts (xy 36.074 252.73) (xy 36.074 249.301))
+  (wire (pts (xy 31.623 253.492) (xy 31.623 250.063))
     (stroke (width 0) (type default))
   )
@@
     (stroke (width 0) (type default))
   )
-  (wire (pts (xy 79.629 40.513) (xy 107.569 40.513))
-    (stroke (width 0) (type default))
-  )
   (bus (pts (xy 110.109 73.533) (xy 110.109 70.993))
     (stroke (width 0) (type default))
@@
     (stroke (width 0) (type default))
   )
-  (wire (pts (xy 79.629 45.593) (xy 107.569 45.593))
-    (stroke (width 0) (type default))
-  )
   (wire (pts (xy 43.44 172.974) (xy 43.44 184.277))
     (stroke (width 0) (type default))
@@
     (stroke (width 0) (type default))
   )
-  (wire (pts (xy 26.041 249.301) (xy 33.534 249.301))
+  (wire (pts (xy 21.59 250.063) (xy 29.083 250.063))
     (stroke (width 0) (type default))
   )
@@
     (stroke (width 0) (type default))
   )
-  (wire (pts (xy 43.821 222.504) (xy 43.821 229.108))
+  (wire (pts (xy 39.37 223.266) (xy 39.37 229.87))
     (stroke (width 0) (type default))
   )
@@
     (stroke (width 0) (type default))
   )
+  (wire (pts (xy 79.629 45.593) (xy 107.569 45.593))
+    (stroke (width 0) (type default))
+  )
   (bus (pts (xy 126.498 232.537) (xy 126.498 235.077))
     (stroke (width 0) (type default))
@@
     (stroke (width 0) (type default))
   )
-  (wire (pts (xy 29.597 202.057) (xy 67.697 202.057))
+  (wire (pts (xy 25.146 202.057) (xy 67.697 202.057))
     (stroke (width 0) (type default))
   )
@@
     (stroke (width 0) (type default))
   )
-  (wire (pts (xy 29.597 222.504) (xy 29.597 202.057))
+  (wire (pts (xy 25.146 223.266) (xy 25.146 202.057))
     (stroke (width 0) (type default))
   )
@@
     (stroke (width 0) (type default))
   )
+  (wire (pts (xy 79.629 40.513) (xy 107.569 40.513))
+    (stroke (width 0) (type default))
+  )
   (wire (pts (xy 48.514 50.673) (xy 54.229 50.673))
     (stroke (width 0) (type default))
@@
     (stroke (width 0) (type default))
   )
-  (wire (pts (xy 39.757 204.597) (xy 39.757 222.504))
+  (wire (pts (xy 35.306 204.597) (xy 35.306 223.266))
     (stroke (width 0) (type default))
   )
@@
     (stroke (width 0) (type default))
   )
-  (wire (pts (xy 36.074 249.301) (xy 43.821 249.301))
+  (wire (pts (xy 31.623 250.063) (xy 39.37 250.063))
     (stroke (width 0) (type default))
   )
@@
     (stroke (width 0) (type default))
   )
-  (wire (pts (xy 79.629 37.973) (xy 107.569 37.973))
-    (stroke (width 0) (type default))
-  )
   (wire (pts (xy 85.1788 53.213) (xy 107.569 53.213))
     (stroke (width 0) (type default))
@@
     (stroke (width 0) (type default))
   )
-  (wire (pts (xy 67.697 204.597) (xy 39.757 204.597))
+  (wire (pts (xy 67.697 204.597) (xy 35.306 204.597))
     (stroke (width 0) (type default))
   )
@@
     (stroke (width 0) (type default))
   )
-  (wire (pts (xy 39.757 222.504) (xy 43.821 222.504))
+  (wire (pts (xy 35.306 223.266) (xy 39.37 223.266))
     (stroke (width 0) (type default))
   )
@@
     (stroke (width 0) (type default))
   )
-  (wire (pts (xy 26.041 249.301) (xy 26.041 236.728))
+  (wire (pts (xy 21.59 250.063) (xy 21.59 237.49))
     (stroke (width 0) (type default))
   )
@@
   )
   (rectangle (start 16.764 116.84) (end 47.117 152.4)
-    (stroke (width 0) (type default))
+    (stroke (width 0.5) (type default))
+    (fill (type none))
+  )
+  (rectangle (start 16.764 233.68) (end 44.196 263.144)
+    (stroke (width 0.5) (type default))
     (fill (type none))
   )
@@
     (effects (font (size 2 2) (thickness 0.8) bold) (justify left bottom))
   )
+  (text "Isolation to Car" (at 45.212 251.206 0)
+    (effects (font (size 2 2) (thickness 0.8) bold) (justify left bottom))
+  )
   (text "Mux set 1" (at 256.286 208.661 0)
     (effects (font (size 1.27 1.27) bold) (justify left bottom))
@@
     )
   )
-  (label "IPA" (at 39.757 249.301 180) (fields_autoplaced)
+  (label "IPA" (at 35.306 250.063 180) (fields_autoplaced)
     (effects (font (size 1.27 1.27)) (justify right bottom))
   )
@@
     (effects (font (size 1.27 1.27)) (justify left bottom))
   )
-  (label "IMA" (at 29.597 249.301 0) (fields_autoplaced)
+  (label "IMA" (at 25.146 250.063 0) (fields_autoplaced)
     (effects (font (size 1.27 1.27)) (justify left bottom))
   )
@@
       (effects (font (size 1.27 1.27)))
     )
-    (property "Value" "100nF" (at 280.289 130.556 90)
+    (property "Value" "15u" (at 280.289 130.556 90)
       (effects (font (size 1.27 1.27)))
     )
@@
     )
   )
-  (symbol (lib_id "Connector_Generic:Conn_01x02") (at 36.074 257.81 270) (unit 1)
-    (in_bom yes) (on_board yes) (dnp no) (fields_autoplaced)
-    (property "Reference" "J1" (at 38.995 256.5399 90)
+  (symbol (lib_id "Connector_Generic:Conn_01x02") (at 31.623 258.572 270) (unit 1)
+    (in_bom yes) (on_board yes) (dnp no)
+    (property "Reference" "J1" (at 34.544 257.3019 90)
       (effects (font (size 1.27 1.27)) (justify left))
     )
-    (property "Value" "Conn_01x02" (at 38.995 259.0799 90)
+    (property "Value" "Conn_01x02" (at 24.892 261.366 90)
       (effects (font (size 1.27 1.27)) (justify left))
     )
-    (property "Footprint" "Connector_JST:JST_XH_S2B-XH-A-1_1x02_P2.50mm_Horizontal" (at 36.074 257.81 0)
+    (property "Footprint" "Connector_JST:JST_XH_S2B-XH-A-1_1x02_P2.50mm_Horizontal" (at 31.623 258.572 0)
       (effects (font (size 1.27 1.27)) hide)
     )
-    (property "Datasheet" "~" (at 36.074 257.81 0)
+    (property "Datasheet" "~" (at 31.623 258.572 0)
       (effects (font (size 1.27 1.27)) hide)
     )
@@
       (effects (font (size 1.27 1.27)))
     )
-    (property "Value" "100nF" (at 272.796 74.295 90)
+    (property "Value" "15u" (at 272.796 74.295 90)
       (effects (font (size 1.27 1.27)))
     )
@@
       (effects (font (size 1.27 1.27)))
     )
-    (property "Value" "100nF" (at 233.172 73.787 90)
+    (property "Value" "15u" (at 233.172 73.787 90)
       (effects (font (size 1.27 1.27)))
     )
@@
       (effects (font (size 1.27 1.27)))
     )
-    (property "Value" "100nF" (at 231.775 200.406 90)
+    (property "Value" "15u" (at 231.775 200.406 90)
       (effects (font (size 1.27 1.27)))
     )
@@
       (effects (font (size 1.27 1.27)))
     )
-    (property "Value" "100nF" (at 226.695 257.302 90)
+    (property "Value" "15u" (at 226.695 257.302 90)
       (effects (font (size 1.27 1.27)))
     )
@@
       (effects (font (size 1.27 1.27)))
     )
-    (property "Value" "100nF" (at 275.082 257.556 90)
+    (property "Value" "15u" (at 275.082 257.556 90)
       (effects (font (size 1.27 1.27)))
     )
@@
       (effects (font (size 1.27 1.27)))
     )
-    (property "Value" "100nF" (at 278.638 199.517 90)
+    (property "Value" "15u" (at 278.638 199.517 90)
       (effects (font (size 1.27 1.27)))
     )
@@
       (effects (font (size 1.27 1.27)))
     )
-    (property "Value" "100nF" (at 235.458 131.699 90)
+    (property "Value" "15u" (at 235.458 131.699 90)
       (effects (font (size 1.27 1.27)))
     )
@@
     )
   )
-  (symbol (lib_id "esmit:ESMIT-4180_C") (at 26.041 229.108 0) (unit 1)
+  (symbol (lib_id "esmit:ESMIT-4180_C") (at 21.59 229.87 0) (unit 1)
     (in_bom yes) (on_board yes) (dnp no) (fields_autoplaced)
-    (property "Reference" "T1" (at 34.931 220.599 0)
+    (property "Reference" "T1" (at 30.48 221.361 0)
       (effects (font (size 1.524 1.524)))
     )
-    (property "Value" "ESMIT-4180_C" (at 34.931 224.409 0)
+    (property "Value" "ESMIT-4180_C" (at 30.48 225.171 0)
       (effects (font (size 1.524 1.524)))
     )
-    (property "Footprint" "AERO_Footprints:SOIC4_CBM4D19_SUM" (at 26.041 229.108 0)
+    (property "Footprint" "AERO_Footprints:SOIC4_CBM4D19_SUM" (at 21.59 229.87 0)
       (effects (font (size 1.27 1.27) italic) hide)
     )
-    (property "Datasheet" "ESMIT-4180/C" (at 26.041 229.108 0)
+    (property "Datasheet" "ESMIT-4180/C" (at 21.59 229.87 0)
       (effects (font (size 1.27 1.27) italic) hide)
     )

Commit message: fixed footy
Parts:
- U10, U9: footprint AERO_Footprints:QFP-64_11x11_Pitch0.5mm -> AERO_Footprints:LTC6812
Changed lines of the file:
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@@
       (effects (font (size 1.27 1.27)) (justify left))
     )
-    (property "Footprint" "AERO_Footprints:QFP-64_11x11_Pitch0.5mm" (at 80.397 194.437 0)
+    (property "Footprint" "AERO_Footprints:LTC6812" (at 80.397 194.437 0)
       (effects (font (size 1.27 1.27)) hide)
     )
@@
       (effects (font (size 1.27 1.27)) (justify left))
     )
-    (property "Footprint" "AERO_Footprints:QFP-64_11x11_Pitch0.5mm" (at 66.929 73.533 0)
-      (effects (font (size 1.27 1.27)) hide)
-    )
+    (property "Footprint" "AERO_Footprints:LTC6812" (at 66.929 73.533 0)
+      (effects (font (size 1.27 1.27)) hide)
+    )

Commit message: final before comp
Parts:
- removed Q1: Q_NPN_BCE, AERO_Footprints:DXT5551P5-13_DIO, symbol Device:Q_NPN_BCE
- added Q3: DXT5551P5-13_DIO, AERO_Footprints:DXT5551P5-13_DIO, symbol Device:Q_NPN_BCE
- added R96: 100, symbol Device:R_US
- Q2: value Q_NPN_BCE -> DXT5551P5-13_DIO
Connections:
- net VCC: now also Q2.1 (C); no longer Q2.2 (C)
- net VDC: now also Q3.1 (C)
- net VDD: now also Q3.3 (E)
- net at U10.49 (DRIVE): now also Q2.2 (B); no longer Q2.1 (B)
- net at T1.1, U10.61 (CSB(IMA)): now also R96.1
- net at T1.2, U10.62 (SCK(IPA)): now also R96.2
- net at U9.49 (DRIVE): now also Q3.2 (B)
Changed lines of the file:
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@@
   (junction (at 43.44 184.277) (diameter 0) (color 0 0 0 0)
   )
+  (junction (at 25.146 214.884) (diameter 0) (color 0 0 0 0)
+  )
   (junction (at 126.498 197.993) (diameter 0) (color 0 0 0 0)
   )
@@
   (junction (at 269.24 44.704) (diameter 0) (color 0 0 0 0)
   )
+  (junction (at 35.306 214.884) (diameter 0) (color 0 0 0 0)
+  )
   (junction (at 266.319 99.568) (diameter 0) (color 0 0 0 0)
   )
@@
     (stroke (width 0) (type default))
   )
+  (wire (pts (xy 25.146 202.057) (xy 25.146 214.884))
+    (stroke (width 0) (type default))
+  )
   (wire (pts (xy 266.319 97.028) (xy 266.319 99.568))
     (stroke (width 0) (type default))
@@
     (stroke (width 0) (type default))
   )
+  (wire (pts (xy 33.909 214.884) (xy 35.306 214.884))
+    (stroke (width 0) (type default))
+  )
   (wire (pts (xy 45.72 24.765) (xy 36.068 24.765))
     (stroke (width 0) (type default))
@@
     (stroke (width 0) (type default))
   )
+  (wire (pts (xy 35.306 214.884) (xy 35.306 223.266))
+    (stroke (width 0) (type default))
+  )
   (wire (pts (xy 102.8839 184.277) (xy 123.958 184.277))
     (stroke (width 0) (type default))
@@
     (stroke (width 0) (type default))
   )
-  (wire (pts (xy 39.37 237.49) (xy 39.37 250.063))
-    (stroke (width 0) (type default))
-  )
   (wire (pts (xy 103.0603 209.677) (xy 123.958 209.677))
     (stroke (width 0) (type default))
@@
     (stroke (width 0) (type default))
   )
+  (wire (pts (xy 26.289 214.884) (xy 25.146 214.884))
+    (stroke (width 0) (type default))
+  )
   (wire (pts (xy 225.552 166.624) (xy 225.552 169.164))
     (stroke (width 0) (type default))
@@
     (stroke (width 0) (type default))
   )
+  (wire (pts (xy 35.306 204.597) (xy 35.306 214.884))
+    (stroke (width 0) (type default))
+  )
   (wire (pts (xy 273.304 190.5) (xy 274.955 190.5))
     (stroke (width 0) (type default))
@@
     (stroke (width 0) (type default))
   )
-  (wire (pts (xy 25.146 223.266) (xy 25.146 202.057))
-    (stroke (width 0) (type default))
-  )
   (polyline (pts (xy 302.006 77.978) (xy 302.006 79.629))
     (stroke (width 0) (type default))
@@
     (stroke (width 0) (type default))
   )
-  (wire (pts (xy 35.306 204.597) (xy 35.306 223.266))
-    (stroke (width 0) (type default))
-  )
   (wire (pts (xy 269.748 170.307) (xy 269.748 170.18))
     (stroke (width 0) (type default))
@@
     (stroke (width 0) (type default))
   )
+  (wire (pts (xy 39.37 237.49) (xy 39.37 250.063))
+    (stroke (width 0) (type default))
+  )
   (wire (pts (xy 272.796 42.164) (xy 269.24 42.164))
     (stroke (width 0) (type default))
@@
     (stroke (width 0) (type default))
   )
+  (wire (pts (xy 21.59 237.49) (xy 21.59 250.063))
+    (stroke (width 0) (type default))
+  )
   (wire (pts (xy 301.498 245.999) (xy 295.275 245.999))
     (stroke (width 0) (type default))
@@
     (stroke (width 0) (type default))
   )
+  (wire (pts (xy 25.146 214.884) (xy 25.146 223.266))
+    (stroke (width 0) (type default))
+  )
   (bus (pts (xy 110.109 83.693) (xy 110.109 81.153))
     (stroke (width 0) (type default))
@@
     (stroke (width 0) (type default))
   )
-  (wire (pts (xy 21.59 250.063) (xy 21.59 237.49))
-    (stroke (width 0) (type default))
-  )
   (wire (pts (xy 93.097 227.457) (xy 123.958 227.457))
     (stroke (width 0) (type default))
@@
     )
   )
-  (symbol (lib_id "Device:Q_NPN_BCE") (at 61.474 146.431 270) (mirror x) (unit 1)
+  (symbol (lib_name "Q_NPN_BCE_1") (lib_id "Device:Q_NPN_BCE") (at 61.474 146.431 270) (mirror x) (unit 1)
     (in_bom yes) (on_board yes) (dnp no) (fields_autoplaced)
     (property "Reference" "Q2" (at 61.474 136.525 90)
       (effects (font (size 1.27 1.27)))
     )
-    (property "Value" "Q_NPN_BCE" (at 61.474 139.065 90)
+    (property "Value" "DXT5551P5-13_DIO" (at 61.474 139.065 90)
       (effects (font (size 1.27 1.27)))
     )
@@
     )
   )
+  (symbol (lib_id "Device:R_US") (at 30.099 214.884 90) (unit 1)
+    (in_bom yes) (on_board yes) (dnp no)
+    (property "Reference" "R96" (at 30.099 210.185 90)
+      (effects (font (size 1.27 1.27)))
+    )
+    (property "Value" "100" (at 30.099 212.09 90)
+      (effects (font (size 1.27 1.27)))
+    )
+    (property "Footprint" "" (at 30.353 213.868 90)
+      (effects (font (size 1.27 1.27)) hide)
+    )
+    (property "Datasheet" "~" (at 30.099 214.884 0)
+      (effects (font (size 1.27 1.27)) hide)
+    )
+    (pin "1")
+    (pin "2")
+    (instances
+      (project "BMS1"
+        (path "/03933f33-7fdb-43de-9d7d-a565cad8a277"
+          (reference "R96") (unit 1)
+        )
+      )
+    )
+  )
   (symbol (lib_id "power:GND2") (at 248.666 130.048 0) (unit 1)
     (in_bom yes) (on_board yes) (dnp no) (fields_autoplaced)
@@
     )
   )
-  (symbol (lib_id "Device:Q_NPN_BCE") (at 50.8 27.305 270) (mirror x) (unit 1)
-    (in_bom yes) (on_board yes) (dnp no) (fields_autoplaced)
-    (property "Reference" "Q1" (at 50.8 17.907 90)
-      (effects (font (size 1.27 1.27)))
-    )
-    (property "Value" "Q_NPN_BCE" (at 50.8 20.447 90)
-      (effects (font (size 1.27 1.27)))
-    )
-    (property "Footprint" "AERO_Footprints:DXT5551P5-13_DIO" (at 53.34 22.225 0)
-      (effects (font (size 1.27 1.27)) hide)
-    )
-    (property "Datasheet" "~" (at 50.8 27.305 0)
-      (effects (font (size 1.27 1.27)) hide)
-    )
-    (pin "1")
-    (pin "2")
-    (pin "3")
-    (instances
-      (project "BMS1"
-        (path "/03933f33-7fdb-43de-9d7d-a565cad8a277"
-          (reference "Q1") (unit 1)
-        )
-      )
-    )
-  )
   (symbol (lib_id "Device:LED") (at 108.712 142.748 180) (unit 1)
     (in_bom yes) (on_board yes) (dnp no) (fields_autoplaced)
@@
         )
       )
+    )
+  )
+  (symbol (lib_name "Q_NPN_BCE_2") (lib_id "Device:Q_NPN_BCE") (at 50.8 27.305 270) (mirror x) (unit 1)
+    (in_bom yes) (on_board yes) (dnp no)
+    (property "Reference" "Q3" (at 50.8 17.907 90)
+      (effects (font (size 1.27 1.27)))
+    )
+    (property "Value" "DXT5551P5-13_DIO" (at 50.8 20.447 90)
+      (effects (font (size 1.27 1.27)))
+    )
+    (property "Footprint" "AERO_Footprints:DXT5551P5-13_DIO" (at 53.34 22.225 0)
+      (effects (font (size 1.27 1.27)) hide)
+    )
+    (property "Datasheet" "~" (at 50.8 27.305 0)
+      (effects (font (size 1.27 1.27)) hide)
+    )
+    (pin "1")
+    (pin "2")
+    (pin "3")
+    (instances
+      (project "BMS1"
+        (path "/03933f33-7fdb-43de-9d7d-a565cad8a277"
+          (reference "Q3") (unit 1)
+        )
+      )
