File: BMS1/BMS1.kicad_sch (KiCad schematic)
At the start: 55 parts, among them J1 Conn_01x02, J2 Conn_01x02, J3 Conn_01x02, Q2 DXT5551P5-13_DIO, Q3 DXT5551P5-13_DIO, T1 ESMIT-4180_C, U1 ADG728, U10 LTC6812-1, U2 ADG728, U3 ADG728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

Commit message: ERC fixes
Parts:
- R12: MPN (none) -> ERJ-3EKF1004V
Connections:
- net VD: now also R10.2, U10.52 (DTEN)
- net at R11.1, R6.2, U10.58 (ICMP): now also C40.2, U10.50 (VREF2)
Other:
- moved on the sheet: C1, C10, C11, C12, C13, C14, C2, C3, C4, C40, C42, C43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

Commit message: ERC error fixes
Parts:
- removed JP1: Jumper_3_Bridged12, Jumper:SolderJumper-3_P1.3mm_Bridged12_RoundedPad1.0x1.5mm_NumberLabels, symbol Jumper:Jumper_3_Bridged12
- U10, U9: footprint AERO_Footprints:LTC6812 -> AERO_Footprints:QFP-64_11x11_Pitch0.5mm
Connections:
- net VCC: now also Q2.2 (C); no longer Q2.1 (C)
- net VDC: now also Q3.2 (C); no longer Q3.1 (C)
- net at U10.49 (DRIVE): now also Q2.1 (B); no longer Q2.2 (B)
- net at U9.49 (DRIVE): now also Q3.1 (B); no longer Q3.2 (B)
Other:
- note added: "IMA (-), IPA (+): ISOSPI all chip info, differentail pair, must have same length=same resistance, close together - add choke: hot side (close to chip) of transformer IBIAS: controls current on ISOSPI interface - resistor calc on datasheet ICMP: reads IBIAS between voltage divider VREF2 (added cap footprint), VREF1: decoupling capacitors, values on data sheet q2: large, big copper plane around pin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"
- note removed: "GPIO 3,4: SPI to muxes GPIO 8,9: each reads cell temp voltage from diff mux IMA (-), IPA (+): ISOSPI all chip info, differentail pair, must have same length=same resistance, close together - add choke: hot side (close to chip) of transformer IMB, IPB: chip communication WDT: watch dog timer - fault when chip isn't fast enough (2s) - not using here IBIAS: controls current on ISOSPI interface - res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"

Commit message: Footprints
Parts:
- C1, C2, C3, C4, C5, C6, C7, C8: footprint Capacitor_SMD:C_0603_1608Metric_Pad1.08x0.95mm_HandSolder -> Capacitor_SMD:C_0603_1608Metric; MPN (none) -> AGC0603X7R101-104KXP
- C10, C9: footprint Capacitor_SMD:C_0805_2012Metric_Pad1.18x1.45mm_HandSolder -> Capacitor_SMD:C_0805_2012Metric; MPN (none) -> AGC0603X7R500-103KNP
- C11, C12: footprint Capacitor_SMD:C_0603_1608Metric_Pad1.08x0.95mm_HandSolder -> Capacitor_SMD:C_0603_1608Metric; MPN (none) -> GRM033R60J105MEA2D
- C13, C14: value 100nf -> 0.1uF; footprint Capacitor_SMD:C_0603_1608Metric_Pad1.08x0.95mm_HandSolder -> Capacitor_SMD:C_0603_1608Metric; MPN (none) -> AGC0603X7R101-104KXP
- C40: value 1uf -> 1uF; footprint (none) -> Capacitor_SMD:C_0603_1608Metric; MPN (none) -> GRM033R60J105MEA2D
- C41, C42, C43: value 1uf -> 1uF; footprint Capacitor_SMD:C_0603_1608Metric_Pad1.08x0.95mm_HandSolder -> Capacitor_SMD:C_0603_1608Metric; MPN (none) -> GRM033R60J105MEA2D
- D1, D2: footprint LED_SMD:LED_0603_1608Metric_Pad1.05x0.95mm_HandSolder -> LED_SMD:LED_0201_0603Metric
- R1, R10, R11, R2, R5, R6: footprint Resistor_SMD:R_0603_1608Metric_Pad0.98x0.95mm_HandSolder -> Resistor_SMD:R_0603_1608Metric; MPN (none) -> RC0201FR-071KL
- R12: footprint Resistor_SMD:R_0603_1608Metric_Pad0.98x0.95mm_HandSolder -> Resistor_SMD:R_0603_1608Metric; MPN ERJ-3EKF1004V -> ERJ-1GNF1004C
- R3, R4, R8, R9: footprint Resistor_SMD:R_0603_1608Metric_Pad0.98x0.95mm_HandSolder -> Resistor_SMD:R_0603_1608Metric; MPN (none) -> RC0201FR-0720KL
- R7: footprint Resistor_SMD:R_0603_1608Metric_Pad0.98x0.95mm_HandSolder -> Resistor_SMD:R_0603_1608Metric; MPN (none) -> ERJ-1GNF1004C
- R94, R95: footprint Resistor_SMD:R_0603_1608Metric_Pad0.98x0.95mm_HandSolder -> Resistor_SMD:R_0603_1608Metric

Commit message: Footprints
Parts:
- C10, C9: MPN AGC0603X7R500-103KNP -> C0805C103K5RACTU
- C11, C12: value 1uf -> 1uF; MPN GRM033R60J105MEA2D -> CL10B105KP8NNNC
- C40, C41, C42, C43: MPN GRM033R60J105MEA2D -> CL10B105KP8NNNC
- J1: MPN (none) -> S2B-XH-A-1
- J2, J3: MPN (none) -> B2B-XH-A
- L1, L2: MPN (none) -> 744232090
- Q2, Q3: MPN (none) -> DXT5551P5-13
- R1, R10, R11, R2, R5, R6: MPN RC0201FR-071KL -> RC0603FR-071KL
- R12, R7: MPN ERJ-1GNF1004C -> ERJ-3EKF1004V
- R3, R4, R8, R9: MPN RC0201FR-0720KL -> ERJ-3EKF2002V
- R94, R95: MPN (none) -> ERA-3AEB331V
- U1, U2, U3, U4, U5, U6, U7, U8: MPN (none) -> ADG728BRUZ-REEL7
- U10, U9: MPN (none) -> LTC6812ILWE-1#3ZZTRPBF
Changed lines of the file:
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@@
 			)
 		)
-		(property "MPN" ""
+		(property "MPN" "ADG728BRUZ-REEL7"
 			(at 243.84 109.22 0)
 			(effects
@@
 			)
 		)
-		(property "MPN" "RC0201FR-071KL"
+		(property "MPN" "RC0603FR-071KL"
 			(at 57.15 182.88 0)
 			(effects
@@
 			)
 		)
-		(property "Datasheet" "https://mm.digikey.com/Volume0/opasdata/d220001/medias/docus/5561/AGC%20Series.pdf"
+		(property "Datasheet" "https://content.kemet.com/datasheets/KEM_C1002_X7R_SMD.pdf"
 			(at 27.94 120.65 0)
 			(effects
@@
 			)
 		)
-		(property "MPN" "AGC0603X7R500-103KNP"
+		(property "MPN" "C0805C103K5RACTU"
 			(at 27.94 120.65 0)
 			(effects
@@
 			)
 		)
-		(property "MPN" "ERJ-1GNF1004C"
+		(property "MPN" "ERJ-3EKF1004V"
 			(at 62.23 190.5 0)
 			(effects
@@
 			)
 		)
-		(property "MPN" "RC0201FR-071KL"
+		(property "MPN" "RC0603FR-071KL"
 			(at 44.45 66.04 0)
 			(effects
@@
 			)
 		)
-		(property "Datasheet" "https://www.yageo.com/upload/media/product/products/datasheet/rchip/PYu-RC_Group_51_RoHS_L_12.pdf"
+		(property "Datasheet" "https://industrial.panasonic.com/cdbs/www-data/pdf/RDA0000/AOA0000C304.pdf"
 			(at 41.91 104.14 0)
 			(effects
@@
 			)
 		)
-		(property "MPN" "RC0201FR-0720KL"
+		(property "MPN" "ERJ-3EKF2002V"
 			(at 41.91 104.14 0)
 			(effects
@@
 			)
 		)
-		(property "MPN" ""
+		(property "MPN" "ADG728BRUZ-REEL7"
 			(at 241.3 177.8 0)
 			(effects
@@
 			)
 		)
-		(property "Datasheet" ""
+		(property "Datasheet" "https://www.analog.com/media/en/technical-documentation/data-sheets/LTC6812-1.pdf"
 			(at 81.28 195.58 0)
 			(effects
@@
 			)
 		)
-		(property "MPN" ""
+		(property "MPN" "LTC6812ILWE-1#3ZZTRPBF"
 			(at 81.28 205.74 0)
 			(effects
@@
 			)
 		)
-		(property "Datasheet" "~"
+		(property "Datasheet" "https://www.diodes.com/assets/Datasheets/DXT5551P5.pdf"
 			(at 60.96 147.32 0)
 			(effects
@@
 			)
 		)
-		(property "MPN" ""
+		(property "MPN" "DXT5551P5-13"
 			(at 60.96 147.32 0)
 			(effects
@@
 			)
 		)
-		(property "Datasheet" "~"
+		(property "Datasheet" "https://www.jst-mfg.com/product/pdf/eng/eXH.pdf"
 			(at 30.48 134.62 0)
 			(effects
@@
 			)
 		)
-		(property "MPN" ""
+		(property "MPN" "B2B-XH-A"
 			(at 30.48 134.62 0)
 			(effects
@@
 			)
 		)
-		(property "Datasheet" ""
+		(property "Datasheet" "https://www.jst-mfg.com/product/pdf/eng/eXH.pdf"
 			(at 33.02 259.08 0)
 			(effects
@@
 			)
 		)
-		(property "MPN" ""
+		(property "MPN" "S2B-XH-A-1"
 			(at 33.02 259.08 0)
 			(effects
@@
 			)
 		)
-		(property "MPN" "RC0201FR-071KL"
+		(property "MPN" "RC0603FR-071KL"
 			(at 34.29 66.04 0)
 			(effects
@@
 			)
 		)
-		(property "Datasheet" "~"
+		(property "Datasheet" "https://www.jst-mfg.com/product/pdf/eng/eXH.pdf"
 			(at 33.02 132.08 0)
 			(effects
@@
 			)
 		)
-		(property "MPN" ""
+		(property "MPN" "B2B-XH-A"
 			(at 33.02 132.08 0)
 			(effects
@@
 			)
 		)
-		(property "Datasheet" "https://search.murata.co.jp/Ceramy/image/img/A01X/G101/ENG/GRM033R60J105MEA2-02.pdf"
+		(property "Datasheet" "https://mm.digikey.com/Volume0/opasdata/d220001/medias/docus/3584/CL10B105KP8NNNC_Spec.pdf"
 			(at 49.53 177.8 0)
 			(effects
@@
 			)
 		)
-		(property "MPN" "GRM033R60J105MEA2D"
+		(property "MPN" "CL10B105KP8NNNC"
 			(at 49.53 177.8 0)
 			(effects
@@
 			)
 		)
-		(property "Datasheet" "~"
+		(property "Datasheet" "https://industrial.panasonic.com/cdbs/www-data/pdf/RDM0000/AOA0000C307.pdf"
 			(at 119.38 146.05 0)
 			(effects
@@
 			)
 		)
-		(property "MPN" ""
+		(property "MPN" "ERA-3AEB331V"
 			(at 119.38 146.05 0)
 			(effects
@@
 			)
 		)
-		(property "MPN" "ERJ-1GNF1004C"
+		(property "MPN" "ERJ-3EKF1004V"
 			(at 49.53 71.12 0)
 			(effects
@@
 			)
 		)
-		(property "Datasheet" "https://www.yageo.com/upload/media/product/products/datasheet/rchip/PYu-RC_Group_51_RoHS_L_12.pdf"
+		(property "Datasheet" "https://industrial.panasonic.com/cdbs/www-data/pdf/RDA0000/AOA0000C304.pdf"
 			(at 41.91 96.52 0)
 			(effects
@@
 			)
 		)
-		(property "MPN" "RC0201FR-0720KL"
+		(property "MPN" "ERJ-3EKF2002V"
 			(at 41.91 96.52 0)
 			(effects
@@
 			)
 		)
-		(property "Datasheet" "https://www.yageo.com/upload/media/product/products/datasheet/rchip/PYu-RC_Group_51_RoHS_L_12.pdf"
+		(property "Datasheet" "https://industrial.panasonic.com/cdbs/www-data/pdf/RDA0000/AOA0000C304.pdf"
 			(at 57.15 228.6 0)
 			(effects
@@
 			)
 		)
-		(property "MPN" "RC0201FR-0720KL"
+		(property "MPN" "ERJ-3EKF2002V"
 			(at 57.15 228.6 0)
 			(effects
@@
 			)
 		)
-		(property "MPN" ""
+		(property "MPN" "744232090"
 			(at 30.48 213.36 0)
 			(effects
@@
 			)
 		)
-		(property "Datasheet" "https://search.murata.co.jp/Ceramy/image/img/A01X/G101/ENG/GRM033R60J105MEA2-02.pdf"
+		(property "Datasheet" "https://mm.digikey.com/Volume0/opasdata/d220001/medias/docus/3584/CL10B105KP8NNNC_Spec.pdf"
 			(at 31.75 33.02 0)
 			(effects
@@
 			)
 		)
-		(property "MPN" "GRM033R60J105MEA2D"
+		(property "MPN" "CL10B105KP8NNNC"
 			(at 31.75 33.02 0)
 			(effects
@@
 			)
 		)
-		(property "MPN" ""
+		(property "MPN" "ADG728BRUZ-REEL7"
 			(at 289.56 109.22 0)
 			(effects
@@
 			)
 		)
-		(property "MPN" ""
+		(property "MPN" "ADG728BRUZ-REEL7"
 			(at 284.48 177.8 0)
 			(effects
@@
 			)
 		)
-		(property "MPN" ""
+		(property "MPN" "ADG728BRUZ-REEL7"
 			(at 236.22 236.22 0)
 			(effects
@@
 			)
 		)
-		(property "MPN" ""
+		(property "MPN" "ADG728BRUZ-REEL7"
 			(at 284.48 236.22 0)
 			(effects
@@
 			)
 		)
-		(property "MPN" ""
+		(property "MPN" "ADG728BRUZ-REEL7"
 			(at 243.84 50.8 0)
 			(effects
@@
 			)
 		)
-		(property "MPN" ""
+		(property "MPN" "744232090"
 			(at 30.48 96.52 0)
 			(effects
@@
 			)
 		)
-		(property "Datasheet" "~"
+		(property "Datasheet" "https://industrial.panasonic.com/cdbs/www-data/pdf/RDM0000/AOA0000C307.pdf"
 			(at 114.3 31.75 0)
 			(effects
@@
 			)
 		)
-		(property "MPN" ""
+		(property "MPN" "ERA-3AEB331V"
 			(at 114.3 31.75 0)
 			(effects
@@
 			)
 		)
-		(property "MPN" "RC0201FR-071KL"
+		(property "MPN" "RC0603FR-071KL"
 			(at 49.53 165.1 0)
 			(effects
@@
 			)
 		)
-		(property "MPN" "RC0201FR-071KL"
+		(property "MPN" "RC0603FR-071KL"
 			(at 39.37 48.26 0)
 			(effects
@@
 			)
 		)
-		(property "Datasheet" "https://search.murata.co.jp/Ceramy/image/img/A01X/G101/ENG/GRM033R60J105MEA2-02.pdf"
+		(property "Datasheet" "https://mm.digikey.com/Volume0/opasdata/d220001/medias/docus/3584/CL10B105KP8NNNC_Spec.pdf"
 			(at 39.37 55.88 0)
 			(effects
@@
 			)
 		)
-		(property "MPN" "GRM033R60J105MEA2D"
+		(property "MPN" "CL10B105KP8NNNC"
 			(at 39.37 55.88 0)
 			(effects
@@
 			)
 		)
-		(property "Datasheet" "https://www.yageo.com/upload/media/product/products/datasheet/rchip/PYu-RC_Group_51_RoHS_L_12.pdf"
+		(property "Datasheet" "https://industrial.panasonic.com/cdbs/www-data/pdf/RDA0000/AOA0000C304.pdf"
 			(at 54.61 223.52 0)
 			(effects
@@
 			)
 		)
-		(property "MPN" "RC0201FR-0720KL"
+		(property "MPN" "ERJ-3EKF2002V"
 			(at 54.61 223.52 0)
 			(effects
@@
 			)
 		)
-		(property "Datasheet" "~"
+		(property "Datasheet" "https://www.diodes.com/assets/Datasheets/DXT5551P5.pdf"
 			(at 50.8 27.94 0)
 			(effects
@@
 			)
 		)
-		(property "MPN" ""
+		(property "MPN" "DXT5551P5-13"
 			(at 50.8 27.94 0)
 			(effects
@@
 			)
 		)
-		(property "Value" "1uf"
+		(property "Value" "1uF"
 			(at 56.896 171.45 90)
 			(effects
@@
 			)
 		)
-		(property "Datasheet" "https://search.murata.co.jp/Ceramy/image/img/A01X/G101/ENG/GRM033R60J105MEA2-02.pdf"
+		(property "Datasheet" "https://mm.digikey.com/Volume0/opasdata/d220001/medias/docus/3584/CL10B105KP8NNNC_Spec.pdf"
 			(at 59.69 170.18 0)
 			(effects
@@
 			)
 		)
-		(property "MPN" "GRM033R60J105MEA2D"
+		(property "MPN" "CL10B105KP8NNNC"
 			(at 59.69 170.18 0)
 			(effects
@@
 			)
 		)
-		(property "Datasheet" ""
+		(property "Datasheet" "https://www.analog.com/media/en/technical-documentation/data-sheets/LTC6812-1.pdf"
 			(at 66.04 73.66 0)
 			(effects
@@
 			)
 		)
-		(property "MPN" ""
+		(property "MPN" "LTC6812ILWE-1#3ZZTRPBF"
 			(at 66.04 83.82 0)
 			(effects
@@
 			)
 		)
-		(property "Value" "1uf"
+		(property "Value" "1uF"
 			(at 44.45 54.61 90)
 			(effects
@@
 			)
 		)
-		(property "Datasheet" "https://search.murata.co.jp/Ceramy/image/img/A01X/G101/ENG/GRM033R60J105MEA2-02.pdf"
+		(property "Datasheet" "https://mm.digikey.com/Volume0/opasdata/d220001/medias/docus/3584/CL10B105KP8NNNC_Spec.pdf"
 			(at 46.99 53.34 0)
 			(effects
@@
 			)
 		)
-		(property "MPN" "GRM033R60J105MEA2D"
+		(property "MPN" "CL10B105KP8NNNC"
 			(at 46.99 53.34 0)
 			(effects
@@
 			)
 		)
-		(property "Datasheet" "https://search.murata.co.jp/Ceramy/image/img/A01X/G101/ENG/GRM033R60J105MEA2-02.pdf"
+		(property "Datasheet" "https://mm.digikey.com/Volume0/opasdata/d220001/medias/docus/3584/CL10B105KP8NNNC_Spec.pdf"
 			(at 52.07 154.94 0)
 			(effects
@@
 			)
 		)
-		(property "MPN" "GRM033R60J105MEA2D"
+		(property "MPN" "CL10B105KP8NNNC"
 			(at 52.07 154.94 0)
 			(effects
@@
 			)
 		)
-		(property "Datasheet" "https://mm.digikey.com/Volume0/opasdata/d220001/medias/docus/5561/AGC%20Series.pdf"
+		(property "Datasheet" "https://content.kemet.com/datasheets/KEM_C1002_X7R_SMD.pdf"
 			(at 35.56 148.59 0)
 			(effects
@@
 			)
 		)
-		(property "MPN" "AGC0603X7R500-103KNP"
+		(property "MPN" "C0805C103K5RACTU"
 			(at 35.56 148.59 0)
 			(effects
@@
 			)
 		)
-		(property "MPN" ""
+		(property "MPN" "ADG728BRUZ-REEL7"
 			(at 281.94 53.34 0)
 			(effects
@@
 			)
 		)
-		(property "MPN" "RC0201FR-071KL"
+		(property "MPN" "RC0603FR-071KL"
 			(at 49.53 187.96 0)
 			(effects
