File: BMS1/BMS1.kicad_pcb (KiCad board)
At the start: 2 copper layers, 122 parts, among them J1 Conn_01x02, U1 ADG728, U10 LTC6812-1, U2 ADG728, U3 ADG728, U4 ADG728, U5 ADG728, U6 ADG728, U7 ADG728, U8 ADG728, U9 LTC6812-1

Commit message: start footprint
Parts:
- removed R90: 680, Resistor_SMD:R_0603_1608Metric_Pad0.98x0.95mm_HandSolder
- added B1: VTC6+T, AERO_Footprints:VTC-6, F.Cu at (104.4, 65.0)
- added B10: VTC6+T, AERO_Footprints:VTC-6, F.Cu at (191.2, 65.0)
- added B11: VTC6+T, AERO_Footprints:VTC-6, F.Cu at (427.0, 65.0)
- added B12: VTC6+T, AERO_Footprints:VTC-6, F.Cu at (19.8, 65.0)
- added B13: VTC6+T, AERO_Footprints:VTC-6, F.Cu at (62.6, 65.0)
- added B14: VTC6+T, AERO_Footprints:VTC-6, F.Cu at (534.1, 65.0)
- added B15: VTC6+T, AERO_Footprints:VTC-6, F.Cu at (298.3, 65.0)
- added B16: VTC6+T, AERO_Footprints:VTC-6, F.Cu at (126.9, 65.0)
- added B17: VTC6+T, AERO_Footprints:VTC-6, F.Cu at (469.8, 65.0)
- added B18: VTC6+T, AERO_Footprints:VTC-6, F.Cu at (341.3, 65.0)
- added B19: VTC6+T, AERO_Footprints:VTC-6, F.Cu at (41.2, 65.0)
- added B2: VTC6+T, AERO_Footprints:VTC-6, F.Cu at (169.7, 65.0)
- added B20: VTC6+T, AERO_Footprints:VTC-6, F.Cu at (212.6, 65.0)
- added B21: VTC6+T, AERO_Footprints:VTC-6, F.Cu at (255.4, 65.0)
- added B22: VTC6+T, AERO_Footprints:VTC-6, F.Cu at (234.0, 65.0)
- added B23: VTC6+T, AERO_Footprints:VTC-6, F.Cu at (491.2, 65.0)
- added B24: VTC6+T, AERO_Footprints:VTC-6, F.Cu at (276.8, 65.0)
- added B25: VTC6+T, AERO_Footprints:VTC-6, F.Cu at (448.4, 65.0)
- added B3: VTC6+T, AERO_Footprints:VTC-6, F.Cu at (405.6, 65.0)
- added B4: VTC6+T, AERO_Footprints:VTC-6, F.Cu at (319.9, 65.0)
- added B5: VTC6+T, AERO_Footprints:VTC-6, F.Cu at (148.3, 65.0)
- added B6: VTC6+T, AERO_Footprints:VTC-6, F.Cu at (84.1, 65.0)
- added B7: VTC6+T, AERO_Footprints:VTC-6, F.Cu at (384.1, 65.0)
- added B8: VTC6+T, AERO_Footprints:VTC-6, F.Cu at (512.7, 65.0)
- added B9: VTC6+T, AERO_Footprints:VTC-6, F.Cu at (362.7, 65.0)
- R10: footprint Resistor_SMD:R_1206_3216Metric_Pad1.30x1.75mm_HandSolder -> Resistor_SMD:R_0603_1608Metric_Pad0.98x0.95mm_HandSolder
- R22: footprint Resistor_SMD:R_0603_1608Metric_Pad0.98x0.95mm_HandSolder -> Resistor_SMD:R_1206_3216Metric_Pad1.30x1.75mm_HandSolder
- moved R63 205.0 mm to (-5.05, -26.1)
- moved R22 202.4 mm to (-14.6, -27.1)
- moved R60 201.8 mm to (-10.1, -50.7)
- moved U7 199.9 mm to (-12.9, -45.5)
- moved R80 199.7 mm to (5.55, -40.0)
- moved R12 199.5 mm to (-32.4, -28.8)
- moved R72 197.2 mm to (-5.10, -31.1)
- moved R53 197.1 mm to (-14.6, -30.4)
- moved R58 197.0 mm to (-5.55, -40.7)
- moved R17 196.9 mm to (-26.4, -27.1)
- moved R87 196.8 mm to (-0.70, -30.2)
- moved R69 196.0 mm to (-3.50, -34.5)
- moved R77 195.2 mm to (-9.40, -26.1)
- moved R18 195.0 mm to (7.70, -50.5)
- moved C18 194.0 mm to (5.20, -32.5)
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Connections:
- net /BatteryBus.C15 renamed /BatteryBus.C14
- net /BatteryBus1.C13 renamed /BatteryBus1.C14
- C10 pad 1: Net-(C10-Pad1) -> /BatteryBus1.C9
- R10 pad 1: Net-(B8-Pad2) -> GND2
- R10 pad 2: /BatteryBus1.C4 -> /BatteryBus1.C0
- R11 pad 1: Net-(B11-Pad2) -> Net-(B8-Pad2)
- R11 pad 2: /BatteryBus1.C1 -> /BatteryBus1.C4
- R12 pad 1: Net-(B1-Pad2) -> Net-(B11-Pad2)
- R12 pad 2: /BatteryBus1.C11 -> /BatteryBus1.C1
- R13 pad 1: Net-(B2-Pad2) -> Net-(B1-Pad2)
- R13 pad 2: /BatteryBus1.C10 -> /BatteryBus1.C11
- R14 pad 1: Net-(B10-Pad2) -> Net-(B2-Pad2)
- R14 pad 2: /BatteryBus1.C2 -> /BatteryBus1.C10
- R15 pad 1: Net-(B1-Pad1) -> Net-(B10-Pad2)
- R15 pad 2: /BatteryBus1.C12 -> /BatteryBus1.C2
- R16 pad 1: Net-(B7-Pad2) -> Net-(B1-Pad1)
- R16 pad 2: /BatteryBus1.C5 -> /BatteryBus1.C12
- R17 pad 1: Net-(B10-Pad1) -> Net-(B7-Pad2)
- R17 pad 2: /BatteryBus1.C3 -> /BatteryBus1.C5
- R18 pad 1: Net-(B3-Pad2) -> Net-(B10-Pad1)
- R18 pad 2: Net-(C10-Pad1) -> /BatteryBus1.C3
- R19 pad 1: Net-(B4-Pad2) -> Net-(B3-Pad2)
- R19 pad 2: /BatteryBus1.C8 -> /BatteryBus1.C9
- R20 pad 1: Net-(B5-Pad2) -> Net-(B4-Pad2)
- R20 pad 2: /BatteryBus1.C7 -> /BatteryBus1.C8
- R21 pad 1: Net-(B6-Pad2) -> Net-(B5-Pad2)
- R21 pad 2: /BatteryBus1.C6 -> /BatteryBus1.C7
- R22 pad 1: GND2 -> Net-(B6-Pad2)
- R22 pad 2: /BatteryBus1.C0 -> /BatteryBus1.C6

Commit message: footy?
Parts:
- moved U10 446.7 mm to (408.2, 64.4)
- moved R31 174.7 mm to (116.0, 52.0), turned to 90 degrees
- moved R1 102.4 mm to (26.8, 51.8), turned to 90 degrees
- moved U9 46.2 mm to (140.4, 64.6)
- moved B14 12.6 mm to (521.6, 63.6)
- moved B8 11.9 mm to (500.8, 63.6)
- moved B23 11.1 mm to (480.2, 63.6)
- moved B17 10.3 mm to (459.6, 63.6)
- moved B25 9.50 mm to (439.0, 63.6)
- moved B11 8.69 mm to (418.4, 63.6)
- moved B3 7.89 mm to (397.8, 63.6)
- moved B12 7.33 mm to (27.0, 63.6)
- moved B7 7.08 mm to (377.2, 63.6)
- moved B19 6.53 mm to (47.6, 63.6)
- moved B9 6.28 mm to (356.6, 63.6)
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
Commit message: footprint
Parts:
- added C32: 100nF, Capacitor_SMD:C_0603_1608Metric_Pad1.08x0.95mm_HandSolder, F.Cu at (573.2, 88.1)
- added C33: 100nF, Capacitor_SMD:C_0603_1608Metric_Pad1.08x0.95mm_HandSolder, F.Cu at (-106.3, 105.4)
- added C34: 100nF, Capacitor_SMD:C_0603_1608Metric_Pad1.08x0.95mm_HandSolder, F.Cu at (-106.3, 65.6)
- added C35: 100nF, Capacitor_SMD:C_0603_1608Metric_Pad1.08x0.95mm_HandSolder, F.Cu at (-106.3, 70.0)
- added C36: 100nF, Capacitor_SMD:C_0603_1608Metric_Pad1.08x0.95mm_HandSolder, F.Cu at (-106.3, 92.1)
- added C37: 100nF, Capacitor_SMD:C_0603_1608Metric_Pad1.08x0.95mm_HandSolder, F.Cu at (-106.3, 127.5)
- added C38: 100nF, Capacitor_SMD:C_0603_1608Metric_Pad1.08x0.95mm_HandSolder, F.Cu at (-106.3, 149.7)
- added C39: 100nF, Capacitor_SMD:C_0603_1608Metric_Pad1.08x0.95mm_HandSolder, F.Cu at (-106.3, 101.0)
- added L1: L_Ferrite_Small, Inductor_SMD:L_0603_1608Metric_Pad1.05x0.95mm_HandSolder, F.Cu at (-53.5, 31.3)
- added L10: L_Ferrite_Small, Inductor_SMD:L_0603_1608Metric_Pad1.05x0.95mm_HandSolder, F.Cu at (-40.0, 47.8)
- added L11: L_Ferrite_Small, Inductor_SMD:L_0603_1608Metric_Pad1.05x0.95mm_HandSolder, F.Cu at (-51.8, 51.2)
- added L12: L_Ferrite_Small, Inductor_SMD:L_0603_1608Metric_Pad1.05x0.95mm_HandSolder, F.Cu at (-40.0, 44.8)
- added L13: L_Ferrite_Small, Inductor_SMD:L_0603_1608Metric_Pad1.05x0.95mm_HandSolder, F.Cu at (-40.0, 41.8)
- added L14: L_Ferrite_Small, Inductor_SMD:L_0603_1608Metric_Pad1.05x0.95mm_HandSolder, F.Cu at (-40.0, 38.8)
- added L15: L_Ferrite_Small, Inductor_SMD:L_0603_1608Metric_Pad1.05x0.95mm_HandSolder, F.Cu at (-52.1, 32.7)
- added L16: L_Ferrite_Small, Inductor_SMD:L_0603_1608Metric_Pad1.05x0.95mm_HandSolder, F.Cu at (-40.0, 35.8)
- added L17: L_Ferrite_Small, Inductor_SMD:L_0603_1608Metric_Pad1.05x0.95mm_HandSolder, F.Cu at (583.6, 106.6)
- added L18: L_Ferrite_Small, Inductor_SMD:L_0603_1608Metric_Pad1.05x0.95mm_HandSolder, F.Cu at (582.1, 105.1)
- added L2: L_Ferrite_Small, Inductor_SMD:L_0603_1608Metric_Pad1.05x0.95mm_HandSolder, F.Cu at (-54.9, 29.9)
- added L20: L_Ferrite_Small, Inductor_SMD:L_0603_1608Metric_Pad1.05x0.95mm_HandSolder, F.Cu at (583.2, 83.1)
- added L21: L_Ferrite_Small, Inductor_SMD:L_0603_1608Metric_Pad1.05x0.95mm_HandSolder, F.Cu at (576.8, 87.6)
- added L23: L_Ferrite_Small, Inductor_SMD:L_0603_1608Metric_Pad1.05x0.95mm_HandSolder, F.Cu at (587.4, 78.9)
- added L24: L_Ferrite_Small, Inductor_SMD:L_0603_1608Metric_Pad1.05x0.95mm_HandSolder, F.Cu at (586.0, 80.3)
- added L25: L_Ferrite_Small, Inductor_SMD:L_0603_1608Metric_Pad1.05x0.95mm_HandSolder, F.Cu at (584.6, 81.7)
- added L26: L_Ferrite_Small, Inductor_SMD:L_0603_1608Metric_Pad1.05x0.95mm_HandSolder, F.Cu at (576.8, 89.6)
- added L27: L_Ferrite_Small, Inductor_SMD:L_0603_1608Metric_Pad1.05x0.95mm_HandSolder, F.Cu at (580.6, 103.6)
- added L28: L_Ferrite_Small, Inductor_SMD:L_0603_1608Metric_Pad1.05x0.95mm_HandSolder, F.Cu at (576.8, 91.6)
- added L29: L_Ferrite_Small, Inductor_SMD:L_0603_1608Metric_Pad1.05x0.95mm_HandSolder, F.Cu at (576.8, 95.5)
- added L3: L_Ferrite_Small, Inductor_SMD:L_0603_1608Metric_Pad1.05x0.95mm_HandSolder, F.Cu at (-54.4, 53.9)
- added L30: L_Ferrite_Small, Inductor_SMD:L_0603_1608Metric_Pad1.05x0.95mm_HandSolder, F.Cu at (576.8, 99.5)
- added L31: L_Ferrite_Small, Inductor_SMD:L_0603_1608Metric_Pad1.05x0.95mm_HandSolder, F.Cu at (576.8, 93.5)
- added L32: L_Ferrite_Small, Inductor_SMD:L_0603_1608Metric_Pad1.05x0.95mm_HandSolder, F.Cu at (576.8, 97.5)
- added L4: L_Ferrite_Small, Inductor_SMD:L_0603_1608Metric_Pad1.05x0.95mm_HandSolder, F.Cu at (-40.0, 53.9)
- added L7: L_Ferrite_Small, Inductor_SMD:L_0603_1608Metric_Pad1.05x0.95mm_HandSolder, F.Cu at (-55.7, 55.2)
- added L8: L_Ferrite_Small, Inductor_SMD:L_0603_1608Metric_Pad1.05x0.95mm_HandSolder, F.Cu at (-53.1, 52.6)
- added L9: L_Ferrite_Small, Inductor_SMD:L_0603_1608Metric_Pad1.05x0.95mm_HandSolder, F.Cu at (-40.0, 50.9)
- added Q1: Q_NPN_BCE, AERO_Footprints:DXT5551P5-13_DIO, F.Cu at (36.7, 43.4)
- added Q2: Q_NPN_BCE, AERO_Footprints:DXT5551P5-13_DIO, F.Cu at (604.2, 94.3)
- added R2: 1k, Resistor_SMD:R_0603_1608Metric_Pad0.98x0.95mm_HandSolder, F.Cu at (-177.1, 82.7)
- added R3: 20k, Resistor_SMD:R_0603_1608Metric_Pad0.98x0.95mm_HandSolder, F.Cu at (-177.1, 129.3)
- added R35: 21, Resistor_SMD:R_2512_6332Metric_Pad1.40x3.35mm_HandSolder, F.Cu at (251.0, 72.6)
- added R4: 20k, Resistor_SMD:R_0603_1608Metric_Pad0.98x0.95mm_HandSolder, F.Cu at (-177.1, 31.4)
- added R5: 1k, Resistor_SMD:R_0603_1608Metric_Pad0.98x0.95mm_HandSolder, F.Cu at (-177.1, 185.3)
- added R6: 1k, Resistor_SMD:R_0603_1608Metric_Pad0.98x0.95mm_HandSolder, F.Cu at (-177.1, 78.0)
- added R7: 1M, Resistor_SMD:R_0603_1608Metric_Pad0.98x0.95mm_HandSolder, F.Cu at (-177.1, 148.0)
- added R76: 21, Resistor_SMD:R_2512_6332Metric_Pad1.40x3.35mm_HandSolder, F.Cu at (415.6, 72.6)
- added R8: 20k, Resistor_SMD:R_0603_1608Metric_Pad0.98x0.95mm_HandSolder, F.Cu at (-177.1, 138.7)
- added R9: 20k, Resistor_SMD:R_0603_1608Metric_Pad0.98x0.95mm_HandSolder, F.Cu at (-177.1, 115.3)
- added R90: 680, Resistor_SMD:R_0603_1608Metric_Pad0.98x0.95mm_HandSolder, F.Cu at (-177.1, 157.3)
- added R91: 680, Resistor_SMD:R_0603_1608Metric_Pad0.98x0.95mm_HandSolder, F.Cu at (-177.1, 143.3)
- added R92: 680, Resistor_SMD:R_0603_1608Metric_Pad0.98x0.95mm_HandSolder, F.Cu at (-177.1, 208.7)
- added R93: 680, Resistor_SMD:R_0603_1608Metric_Pad0.98x0.95mm_HandSolder, F.Cu at (-177.1, 171.3)
- added T1: ESMIT-4180_C, AERO_Footprints:SOIC4_CBM4D19_SUM, F.Cu at (600.6, 77.0)
- C1, C2: value 10nF -> 100nF
- C10, C9: value 100nF -> 10nF
- C11, C12: value 100nF -> 1uf
- C13, C14: value 100nF -> 100nf
- C3, C4: value 1uf -> 100nF
- C5, C6: value 100nf -> 100nF
- R1: footprint Resistor_SMD:R_2512_6332Metric_Pad1.40x3.35mm_HandSolder -> Resistor_SMD:R_0603_1608Metric_Pad0.98x0.95mm_HandSolder
- R10: value 10 -> 1k
- R11: value 10 -> 1k; footprint Resistor_SMD:R_1206_3216Metric_Pad1.30x1.75mm_HandSolder -> Resistor_SMD:R_0603_1608Metric_Pad0.98x0.95mm_HandSolder
- R12: value 10 -> 1M; footprint Resistor_SMD:R_1206_3216Metric_Pad1.30x1.75mm_HandSolder -> Resistor_SMD:R_0603_1608Metric_Pad0.98x0.95mm_HandSolder
- R13: value 10 -> 100; footprint Resistor_SMD:R_1206_3216Metric_Pad1.30x1.75mm_HandSolder -> Resistor_SMD:R_0805_2012Metric_Pad1.20x1.40mm_HandSolder
- R14, R15, R16, R17, R18, R19, R20, R21, R22, R52, R53, R55, R56, R57, R58, R59, R60, R61: footprint Resistor_SMD:R_1206_3216Metric_Pad1.30x1.75mm_HandSolder -> Resistor_SMD:R_0805_2012Metric_Pad1.20x1.40mm_HandSolder
- R23, R24, R25, R26: value 21 -> 10; footprint Resistor_SMD:R_2512_6332Metric_Pad1.40x3.35mm_HandSolder -> Resistor_SMD:R_0805_2012Metric_Pad1.20x1.40mm_HandSolder
- R36, R37, R38, R77, R78, R79: value 680 -> 21; footprint Resistor_SMD:R_0603_1608Metric_Pad0.98x0.95mm_HandSolder -> Resistor_SMD:R_2512_6332Metric_Pad1.40x3.35mm_HandSolder
- R39, R80: value 680 -> 100
- R48, R49, R51: value 10 -> 680; footprint Resistor_SMD:R_1206_3216Metric_Pad1.30x1.75mm_HandSolder -> Resistor_SMD:R_0603_1608Metric_Pad0.98x0.95mm_HandSolder
- R50: value 100 -> 680
- R54: value 10 -> 100; footprint Resistor_SMD:R_1206_3216Metric_Pad1.30x1.75mm_HandSolder -> Resistor_SMD:R_0603_1608Metric_Pad0.98x0.95mm_HandSolder
- R62: footprint Resistor_SMD:R_0603_1608Metric_Pad0.98x0.95mm_HandSolder -> Resistor_SMD:R_0805_2012Metric_Pad1.20x1.40mm_HandSolder
- R63, R64, R65, R66: value 21 -> 10; footprint Resistor_SMD:R_0603_1608Metric_Pad0.98x0.95mm_HandSolder -> Resistor_SMD:R_0805_2012Metric_Pad1.20x1.40mm_HandSolder
- R67, R68, R69, R70, R71, R72, R73, R74, R75: footprint Resistor_SMD:R_0603_1608Metric_Pad0.98x0.95mm_HandSolder -> Resistor_SMD:R_2512_6332Metric_Pad1.40x3.35mm_HandSolder
- moved J1 660.1 mm to (612.0, 78.2), turned to 90 degrees
- moved R53 608.8 mm to (577.9, 109.5), turned to 45 degrees
- moved R79 601.9 mm to (613.6, 63.2), turned to -90 degrees
- moved R58 599.9 mm to (583.3, 73.9), turned to -45 degrees
- moved R60 595.9 mm to (567.6, 95.7)
- moved R55 591.3 mm to (579.8, 77.4), turned to -45 degrees
- moved R66 590.5 mm to (579.7, 111.1), turned to 45 degrees
- moved R52 588.9 mm to (567.6, 98.1)
- moved R61 586.1 mm to (567.6, 100.6)
- moved R57 584.8 mm to (576.2, 107.8), turned to 45 degrees
- moved R63 584.0 mm to (567.6, 88.3)
- moved C31 582.2 mm to (571.0, 84.9), turned to 90 degrees
- moved R65 581.1 mm to (567.6, 93.2)
- moved R56 580.2 mm to (578.1, 79.1), turned to -45 degrees
- moved R59 573.6 mm to (581.5, 75.7), turned to -45 degrees
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Connections:
- C1 pad 1: Net-(C1-Pad1) -> GND2
- C1 pad 2: Net-(C1-Pad2) -> VDD
- C10 pad 1: /BatteryBus1.C9 -> Net-(C10-Pad1)
- C10 pad 2: GND -> Net-(C10-Pad2)
- C11 pad 1: /BatteryBus1.C8 -> GND2
- C11 pad 2: GND -> Net-(C11-Pad2)
- C12 pad 1: /BatteryBus1.C7 -> GND1
- C12 pad 2: GND -> Net-(C12-Pad2)
- C13 pad 1: /BatteryBus1.C6 -> VDC
- C14 pad 1: /BatteryBus1.C5 -> VCC
- C15 pad 1: /BatteryBus1.C4 -> /BatteryBus1.C12
- C15 pad 2: GND -> GND2
- C16 pad 1: /BatteryBus1.C3 -> /BatteryBus1.C11
- C16 pad 2: GND -> GND2
- C17 pad 1: /BatteryBus1.C2 -> /BatteryBus1.C10
- C17 pad 2: GND -> GND2
- C18 pad 1: /BatteryBus1.C1 -> /BatteryBus1.C9
- C18 pad 2: GND -> GND2
- C19 pad 1: /BatteryBus.C13 -> /BatteryBus1.C8
- C19 pad 2: GND -> GND2
- C2 pad 1: Net-(C2-Pad1) -> GND1
- C2 pad 2: Net-(C2-Pad2) -> VD
- C20 pad 1: /BatteryBus.C12 -> /BatteryBus1.C7
- C20 pad 2: GND -> GND2
- C21 pad 1: /BatteryBus.C11 -> /BatteryBus1.C6
- C21 pad 2: GND -> GND2
- C22 pad 1: /BatteryBus.C10 -> /BatteryBus1.C5
- C22 pad 2: GND -> GND2
- C23 pad 1: /BatteryBus.C9 -> /BatteryBus1.C4
- C23 pad 2: GND -> GND2
- C24 pad 1: /BatteryBus.C8 -> /BatteryBus1.C3
- C24 pad 2: GND -> GND2
- C25 pad 1: /BatteryBus.C7 -> /BatteryBus1.C2
- C25 pad 2: GND -> GND2
- C26 pad 1: /BatteryBus.C6 -> /BatteryBus1.C1
- C26 pad 2: GND -> GND2
- C27 pad 1: /BatteryBus.C5 -> /BatteryBus.C13
- C27 pad 2: GND -> GND1
- C28 pad 1: /BatteryBus.C4 -> /BatteryBus.C12
- C28 pad 2: GND -> GND1
- C29 pad 1: /BatteryBus.C3 -> /BatteryBus.C11
- C29 pad 2: GND -> GND1
- C3 pad 1: GND1 -> GND2
- C3 pad 2: Net-(C3-Pad2) -> VDD
- C30 pad 1: /BatteryBus.C2 -> /BatteryBus.C10
- C30 pad 2: GND -> GND1
- C31 pad 1: /BatteryBus.C1 -> /BatteryBus.C9
- C31 pad 2: GND -> GND1
- C4 pad 1: GND2 -> GND1
- C4 pad 2: Net-(C4-Pad2) -> VD
- C5 pad 1: VDC -> GND2
- C5 pad 2: GND -> VDD
- C6 pad 1: VCC -> GND1
- C6 pad 2: GND -> VD
- C7 pad 1: /BatteryBus1.C12 -> GND2
- C7 pad 2: GND -> VDD
- C8 pad 1: /BatteryBus1.C11 -> GND1
- C8 pad 2: GND -> VD
- C9 pad 1: /BatteryBus1.C10 -> Net-(C9-Pad1)
- C9 pad 2: GND -> Net-(C9-Pad2)
- R10 pad 1: GND2 -> GND1
- R10 pad 2: /BatteryBus1.C0 -> Net-(R10-Pad2)
- R11 pad 1: Net-(B8-Pad2) -> Net-(R11-Pad1)
- R11 pad 2: /BatteryBus1.C4 -> Net-(R11-Pad2)
- R12 pad 1: Net-(B11-Pad2) -> VD
- R12 pad 2: /BatteryBus1.C1 -> Net-(R12-Pad2)
- R13 pad 1: Net-(B1-Pad2) -> /BatteryBus1.C13
- R13 pad 2: /BatteryBus1.C11 -> Net-(B1-Pad1)
- R14 pad 1: Net-(B2-Pad2) -> GND2
- R14 pad 2: /BatteryBus1.C10 -> /BatteryBus1.C0
- R15 pad 1: Net-(B10-Pad2) -> Net-(B8-Pad2)
- R15 pad 2: /BatteryBus1.C2 -> /BatteryBus1.C4
- R16 pad 1: Net-(B1-Pad1) -> Net-(B11-Pad2)
- R16 pad 2: /BatteryBus1.C12 -> /BatteryBus1.C1
- R17 pad 1: Net-(B7-Pad2) -> Net-(B1-Pad2)
- R17 pad 2: /BatteryBus1.C5 -> /BatteryBus1.C11
- R18 pad 1: Net-(B10-Pad1) -> Net-(B2-Pad2)
- R18 pad 2: /BatteryBus1.C3 -> /BatteryBus1.C10
- R19 pad 1: Net-(B3-Pad2) -> Net-(B10-Pad2)
- R19 pad 2: /BatteryBus1.C9 -> /BatteryBus1.C2
- R20 pad 1: Net-(B4-Pad2) -> Net-(B1-Pad1)
- R20 pad 2: /BatteryBus1.C8 -> /BatteryBus1.C12
- R21 pad 1: Net-(B5-Pad2) -> Net-(B7-Pad2)
- R21 pad 2: /BatteryBus1.C7 -> /BatteryBus1.C5
- R22 pad 1: Net-(B6-Pad2) -> Net-(B10-Pad1)
- R22 pad 2: /BatteryBus1.C6 -> /BatteryBus1.C3
- R23 pad 1: Net-(B1-Pad2) -> Net-(B3-Pad2)
- R23 pad 2: /BatteryBus1.S11 -> /BatteryBus1.C9
- R24 pad 1: Net-(B8-Pad2) -> Net-(B4-Pad2)
- R24 pad 2: /BatteryBus1.S4 -> /BatteryBus1.C8
- R25 pad 1: Net-(B11-Pad2) -> Net-(B5-Pad2)
- R25 pad 2: /BatteryBus1.S1 -> /BatteryBus1.C7
- R26 pad 1: Net-(B2-Pad2) -> Net-(B6-Pad2)
- R26 pad 2: /BatteryBus1.S10 -> /BatteryBus1.C6
- R27 pad 1: Net-(B7-Pad2) -> Net-(B1-Pad2)
- R27 pad 2: /BatteryBus1.S5 -> /BatteryBus1.S11
- R28 pad 1: Net-(B1-Pad1) -> Net-(B8-Pad2)
- R28 pad 2: /BatteryBus1.S12 -> /BatteryBus1.S4
- R29 pad 1: Net-(B3-Pad2) -> Net-(B11-Pad2)
- R29 pad 2: /BatteryBus1.S9 -> /BatteryBus1.S1
- R30 pad 1: Net-(B4-Pad2) -> Net-(B2-Pad2)
- R30 pad 2: /BatteryBus1.S8 -> /BatteryBus1.S10
- R31 pad 1: Net-(B10-Pad2) -> Net-(B7-Pad2)
- R31 pad 2: /BatteryBus1.S2 -> /BatteryBus1.S5
- R32 pad 1: Net-(B5-Pad2) -> Net-(B1-Pad1)
- R32 pad 2: /BatteryBus1.S7 -> /BatteryBus1.S12
- R33 pad 1: Net-(B10-Pad1) -> Net-(B3-Pad2)
- R33 pad 2: /BatteryBus1.S3 -> /BatteryBus1.S9
- R34 pad 1: Net-(B6-Pad2) -> Net-(B4-Pad2)
- R34 pad 2: /BatteryBus1.S6 -> /BatteryBus1.S8
- R36 pad 1: /CT212 -> Net-(B5-Pad2)
- R36 pad 2: /C+212 -> /BatteryBus1.S7
- R37 pad 1: /CT211 -> Net-(B10-Pad1)
- R37 pad 2: /C+211 -> /BatteryBus1.S3
- R38 pad 1: /CT210 -> Net-(B6-Pad2)
- R38 pad 2: /C+210 -> /BatteryBus1.S6
- R39 pad 1: /CT209 -> VDC
- R39 pad 2: /C+209 -> Net-(B1-Pad1)
- R40 pad 1: /CT208 -> /CT212
- R40 pad 2: /C+208 -> /C+212
- R41 pad 1: /CT207 -> /CT211
- R41 pad 2: /C+207 -> /C+211
- R42 pad 1: /CT206 -> /CT210
- R42 pad 2: /C+206 -> /C+210
- R43 pad 1: /CT205 -> /CT209
- R43 pad 2: /C+205 -> /C+209
- R44 pad 1: /CT204 -> /CT208
- R44 pad 2: /C+204 -> /C+208
- R45 pad 1: /CT203 -> /CT207
- R45 pad 2: /C+203 -> /C+207
- R46 pad 1: /CT202 -> /CT206
- R46 pad 2: /C+202 -> /C+206
- R47 pad 1: /CT201 -> /CT205
- R47 pad 2: /C+201 -> /C+205
- R48 pad 1: Net-(B21-Pad2) -> /CT204
- R48 pad 2: /BatteryBus.C4 -> /C+204
- R49 pad 1: Net-(B24-Pad2) -> /CT203
- R49 pad 2: /BatteryBus.C1 -> /C+203
- R50 pad 1: /BatteryBus.C14 -> /CT202
- R50 pad 2: Net-(B13-Pad1) -> /C+202
- R51 pad 1: Net-(B14-Pad2) -> /CT201
- R51 pad 2: /BatteryBus.C11 -> /C+201
- R52 pad 1: Net-(B15-Pad2) -> Net-(B21-Pad2)
- R52 pad 2: /BatteryBus.C10 -> /BatteryBus.C4
- R53 pad 1: Net-(B23-Pad2) -> Net-(B24-Pad2)
- R53 pad 2: /BatteryBus.C2 -> /BatteryBus.C1
- R54 pad 1: Net-(B13-Pad1) -> /BatteryBus.C15
- R54 pad 2: /BatteryBus.C13 -> Net-(B13-Pad1)
- R55 pad 1: Net-(B13-Pad2) -> Net-(B14-Pad2)
- R55 pad 2: /BatteryBus.C12 -> /BatteryBus.C11
- R56 pad 1: Net-(B20-Pad2) -> Net-(B15-Pad2)
- R56 pad 2: /BatteryBus.C5 -> /BatteryBus.C10
- R57 pad 1: Net-(B22-Pad2) -> Net-(B23-Pad2)
- R57 pad 2: /BatteryBus.C3 -> /BatteryBus.C2
- R58 pad 1: Net-(B16-Pad2) -> Net-(B13-Pad1)
- R58 pad 2: /BatteryBus.C9 -> /BatteryBus.C13
- R59 pad 1: Net-(B17-Pad2) -> Net-(B13-Pad2)
- R59 pad 2: /BatteryBus.C8 -> /BatteryBus.C12
- R60 pad 1: Net-(B18-Pad2) -> Net-(B20-Pad2)
- R60 pad 2: /BatteryBus.C7 -> /BatteryBus.C5
- R61 pad 1: Net-(B19-Pad2) -> Net-(B22-Pad2)
- R61 pad 2: /BatteryBus.C6 -> /BatteryBus.C3
- R62 pad 1: GND1 -> Net-(B16-Pad2)
- R62 pad 2: /BatteryBus.C0 -> /BatteryBus.C9
- R63 pad 1: Net-(B14-Pad2) -> Net-(B17-Pad2)
- R63 pad 2: /BatteryBus.S11 -> /BatteryBus.C8
- R64 pad 1: Net-(B21-Pad2) -> Net-(B18-Pad2)
- R64 pad 2: /BatteryBus.S4 -> /BatteryBus.C7
- R65 pad 1: Net-(B24-Pad2) -> Net-(B19-Pad2)
- R65 pad 2: /BatteryBus.S1 -> /BatteryBus.C6
- R66 pad 1: Net-(B15-Pad2) -> GND1
- R66 pad 2: /BatteryBus.S10 -> /BatteryBus.C0
- R67 pad 1: Net-(B20-Pad2) -> Net-(B14-Pad2)
- R67 pad 2: /BatteryBus.S5 -> /BatteryBus.S11
- R68 pad 1: Net-(B13-Pad2) -> Net-(B21-Pad2)
- R68 pad 2: /BatteryBus.S12 -> /BatteryBus.S4
- R69 pad 1: Net-(B16-Pad2) -> Net-(B24-Pad2)
- R69 pad 2: /BatteryBus.S9 -> /BatteryBus.S1
- R70 pad 1: Net-(B17-Pad2) -> Net-(B15-Pad2)
- R70 pad 2: /BatteryBus.S8 -> /BatteryBus.S10
- R71 pad 1: Net-(B23-Pad2) -> Net-(B20-Pad2)
- R71 pad 2: /BatteryBus.S2 -> /BatteryBus.S5
- R72 pad 1: Net-(B18-Pad2) -> Net-(B13-Pad2)
- R72 pad 2: /BatteryBus.S7 -> /BatteryBus.S12
- R73 pad 1: Net-(B22-Pad2) -> Net-(B16-Pad2)
- R73 pad 2: /BatteryBus.S3 -> /BatteryBus.S9
- R74 pad 1: Net-(B19-Pad2) -> Net-(B17-Pad2)
- R74 pad 2: /BatteryBus.S6 -> /BatteryBus.S8
- R75 pad 1: Net-(B13-Pad1) -> Net-(B23-Pad2)
- R75 pad 2: /BatteryBus.S13 -> /BatteryBus.S2
- R77 pad 1: /CT113 -> Net-(B22-Pad2)
- R77 pad 2: /C+113 -> /BatteryBus.S3
- R78 pad 1: /CT112 -> Net-(B19-Pad2)
- R78 pad 2: /C+112 -> /BatteryBus.S6
- R79 pad 1: /CT111 -> Net-(B13-Pad1)
- R79 pad 2: /C+111 -> /BatteryBus.S13
- R80 pad 1: /CT110 -> VCC
- R80 pad 2: /C+110 -> Net-(B13-Pad1)
- R81 pad 1: /CT109 -> /CT113
- R81 pad 2: /C+109 -> /C+113
- R82 pad 1: /CT108 -> /CT112
- R82 pad 2: /C+108 -> /C+112
- R83 pad 1: /CT107 -> /CT111
- R83 pad 2: /C+107 -> /C+111
- R84 pad 1: /CT106 -> /CT110
- R84 pad 2: /C+106 -> /C+110
- R85 pad 1: /CT105 -> /CT109
- R85 pad 2: /C+105 -> /C+109
- R86 pad 1: /CT104 -> /CT108
- R86 pad 2: /C+104 -> /C+108
- R87 pad 1: /CT103 -> /CT107
- R87 pad 2: /C+103 -> /C+107
- R88 pad 1: /CT102 -> /CT106
- R88 pad 2: /C+102 -> /C+106
- R89 pad 1: /CT101 -> /CT105
- R89 pad 2: /C+101 -> /C+105
- U10 pad 10: /BatteryBus.C12 -> Net-(L24-Pad2)
- U10 pad 12: /BatteryBus.C11 -> Net-(L25-Pad2)
- U10 pad 16: /BatteryBus.C10 -> Net-(L20-Pad2)
- U10 pad 18: /BatteryBus.C9 -> Net-(L21-Pad2)
- U10 pad 20: /BatteryBus.C8 -> Net-(L26-Pad2)
- U10 pad 22: /BatteryBus.C7 -> Net-(L28-Pad2)
- U10 pad 24: /BatteryBus.C6 -> Net-(L31-Pad2)
- U10 pad 28: /BatteryBus.C5 -> Net-(L29-Pad2)
- U10 pad 30: /BatteryBus.C4 -> Net-(L32-Pad2)
- U10 pad 32: /BatteryBus.C3 -> Net-(L30-Pad2)
- U10 pad 34: /BatteryBus.C2 -> Net-(L27-Pad2)
- U10 pad 36: /BatteryBus.C1 -> Net-(L18-Pad2)
- U10 pad 38: /BatteryBus.C0 -> Net-(L17-Pad2)
- U10 pad 4: /BatteryBus.C14 -> /BatteryBus.C15
- U10 pad 49: unconnected-(U10-Pad49) -> Net-(Q2-Pad1)
- U10 pad 51: Net-(C3-Pad2) -> Net-(C12-Pad2)
- U10 pad 52: unconnected-(U10-Pad52) -> Net-(R10-Pad2)
- U10 pad 56: unconnected-(U10-Pad56) -> Net-(R12-Pad2)
- U10 pad 57: Net-(R8-Pad2) -> Net-(R11-Pad2)
- U10 pad 58: Net-(R2-Pad2) -> Net-(R11-Pad1)
- U10 pad 6: /BatteryBus.C14 -> /BatteryBus.C15
- U10 pad 63: Net-(C2-Pad2) -> Net-(C10-Pad2)
- U10 pad 64: Net-(C1-Pad2) -> Net-(C9-Pad2)
- U10 pad 8: /BatteryBus.C13 -> Net-(L23-Pad2)
- U9 pad 10: /BatteryBus1.C12 -> Net-(L3-Pad2)
- U9 pad 12: /BatteryBus1.C11 -> Net-(L8-Pad2)
- U9 pad 16: /BatteryBus1.C10 -> Net-(L11-Pad2)
- U9 pad 18: /BatteryBus1.C9 -> Net-(L4-Pad2)
- U9 pad 20: /BatteryBus1.C8 -> Net-(L9-Pad2)
- U9 pad 22: /BatteryBus1.C7 -> Net-(L10-Pad2)
- U9 pad 24: /BatteryBus1.C6 -> Net-(L12-Pad2)
- U9 pad 28: /BatteryBus1.C5 -> Net-(L13-Pad2)
- U9 pad 30: /BatteryBus1.C4 -> Net-(L14-Pad2)
- U9 pad 32: /BatteryBus1.C3 -> Net-(L16-Pad2)
- U9 pad 34: /BatteryBus1.C2 -> Net-(L15-Pad2)
- U9 pad 36: /BatteryBus1.C1 -> Net-(L1-Pad2)
- U9 pad 38: /BatteryBus1.C0 -> Net-(L2-Pad2)
- U9 pad 4: /BatteryBus1.C14 -> /BatteryBus1.C13
- U9 pad 49: unconnected-(U9-Pad49) -> Net-(Q1-Pad1)
- U9 pad 51: Net-(C4-Pad2) -> Net-(C11-Pad2)
- U9 pad 52: unconnected-(U9-Pad52) -> Net-(R2-Pad2)
- U9 pad 56: unconnected-(U9-Pad56) -> Net-(R7-Pad2)
- U9 pad 6: /BatteryBus1.C14 -> /BatteryBus1.C13
- U9 pad 61: Net-(C2-Pad1) -> Net-(C10-Pad1)
- U9 pad 62: Net-(C1-Pad1) -> Net-(C9-Pad1)
- U9 pad 8: /BatteryBus1.C14 -> Net-(L7-Pad2)
Routing:
- net Net-(L7-Pad2): track 0.00 -> 7.96 mm
- net Net-(L3-Pad2): track 0.00 -> 6.78 mm
- net Net-(L2-Pad2): track 0.00 -> 6.56 mm
- net Net-(L8-Pad2): track 0.00 -> 5.59 mm
- net Net-(L1-Pad2): track 0.00 -> 5.34 mm
- net Net-(L15-Pad2): track 0.00 -> 4.65 mm
- net /BatteryBus.C1: track 0.00 -> 4.28 mm
- net /BatteryBus.C2: track 0.00 -> 4.22 mm
- net /BatteryBus.C0: track 0.00 -> 4.21 mm
- net Net-(L11-Pad2): track 0.00 -> 3.99 mm
- net /BatteryBus1.C10: track 0.00 -> 3.55 mm
- net /BatteryBus1.C13: track 0.00 -> 3.10 mm
- net /BatteryBus1.C11: track 0.00 -> 3.04 mm
- net /BatteryBus1.C12: track 0.00 -> 2.98 mm
- net /BatteryBus1.C1: track 0.00 -> 2.54 mm
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Other:
- board outline added: 601.2 x 67.2 mm
- board text added: "7.5 x 5.75"
- board text added: "Isolation"

Commit message: SChematic to sheets
Parts:
- moved R4 448.4 mm to (271.3, 27.0), turned to -90 degrees
- moved R84 443.8 mm to (266.6, 27.0), turned to -90 degrees
- moved R85 439.3 mm to (262.0, 27.0), turned to -90 degrees
- moved R45 434.8 mm to (257.3, 27.0), turned to -90 degrees
- moved R41 430.4 mm to (252.7, 27.0), turned to -90 degrees
- moved R81 426.0 mm to (248.0, 27.0), turned to -90 degrees
- moved R50 421.7 mm to (243.3, 27.0), turned to -90 degrees
- moved R47 417.4 mm to (238.7, 27.0), turned to -90 degrees
- moved R89 413.2 mm to (234.0, 27.0), turned to -90 degrees
- moved R48 409.1 mm to (229.3, 27.0), turned to -90 degrees
- moved R6 405.0 mm to (224.7, 27.0), turned to -90 degrees
- moved R2 401.0 mm to (220.0, 27.0), turned to -90 degrees
- moved R44 397.0 mm to (215.3, 27.0), turned to -90 degrees
- moved R10 393.2 mm to (210.7, 27.0), turned to -90 degrees
- moved R54 389.4 mm to (206.0, 27.0), turned to -90 degrees
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Other:
- board text removed: "7.5 x 5.75"

Commit message: Vias it is
Parts:
- moved R79 34.7 mm to (616.2, 47.8)
- moved J1 12.3 mm to (647.2, 66.0)
- moved T1 12.3 mm to (635.8, 64.8)
- moved R15 1.59 mm to (73.2, 83.9)
- moved R21 1.59 mm to (73.2, 87.2)
- moved R24 1.59 mm to (73.2, 97.0)
- moved R25 1.59 mm to (73.2, 93.7)
- moved L10 1.59 mm to (60.6, 93.2)
- moved L12 1.59 mm to (60.6, 90.2)
- moved L13 1.59 mm to (60.6, 87.2)
- moved L14 1.59 mm to (60.6, 84.2)
- moved L16 1.59 mm to (60.6, 81.2)
- moved L4 1.59 mm to (60.6, 99.3)
- moved L9 1.59 mm to (60.6, 96.3)
- moved R22 1.59 mm to (73.2, 80.6)
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Routing:
- net GND2: track 0.00 -> 268.9 mm
- net Net-(B11-Pad2): track 0.00 -> 260.3 mm
- net Net-(B10-Pad2): track 0.00 -> 238.2 mm
Other:
- board size 601.2 x 67.2 mm -> 625.6 x 67.2 mm

Commit message: Post Design Review
Routing:
- net GND2: track 268.9 -> 7.52 mm
- net Net-(B11-Pad2): track 260.3 -> 0.00 mm
- net Net-(B10-Pad2): track 238.2 -> 0.00 mm
- net Net-(B8-Pad2): track 0.00 -> 164.8 mm, vias 0 -> 1
Changed lines of the file:
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@@
     (pts (xy 649.92 58.6) (xy 649.92 125.8))
     (height -20.2)
-    (gr_text "2.6457 in" (at 668.32 92.2 90) (layer "F.Cu")
+    (gr_text "67.2000 mm" (at 668.32 92.2 90) (layer "F.Cu")
       (effects (font (size 1.5 1.5) (thickness 0.3)))
     )
@@
     (pts (xy 23.876 125.476) (xy 649.732 125.468001))
     (height 13.723999)
-    (gr_text "24.6400 in" (at 336.804152 137.395999 0.0007323829061) (layer "F.SilkS")
+    (gr_text "625.8560 mm" (at 336.804152 137.395999 0.0007323829061) (layer "F.SilkS")
       (effects (font (size 1.5 1.5) (thickness 0.3)))
     )
@@
     (style (thickness 0.2) (arrow_length 1.27) (text_position_mode 0) (extension_height 0.58642) (extension_offset 0.5) keep_text_aligned)
   )
+  (segment (start 78.74 83.82) (end 78.683468 83.876532) (width 0.25) (layer "F.Cu") (net 1))
+  (segment (start 78.683468 83.876532) (end 74.152 83.876532) (width 0.25) (layer "F.Cu") (net 1))
+  (via (at 78.74 83.82) (size 0.8) (drill 0.4) (layers "F.Cu" "B.Cu") (net 1))
+  (segment (start 219 83.82) (end 78.74 83.82) (width 0.25) (layer "B.Cu") (net 1))
+  (segment (start 233.12 69.7) (end 219 83.82) (width 0.25) (layer "B.Cu") (net 1))
   (segment (start 49.777071 76.039729) (end 48.218716 77.598084) (width 0.25) (layer "F.Cu") (net 2))
   (segment (start 49.777071 75.993874) (end 49.777071 76.039729) (width 0.25) (layer "F.Cu") (net 2))
   (segment (start 48.090497 77.389013) (end 48.381932 77.389013) (width 0.25) (layer "F.Cu") (net 2))
-  (segment (start 51.191285 74.57966) (end 79.509486 74.57966) (width 0.25) (layer "F.Cu") (net 3))
-  (segment (start 79.509486 74.57966) (end 93.004826 88.075) (width 0.25) (layer "F.Cu") (net 3))
-  (segment (start 220.155 88.075) (end 241.3 109.22) (width 0.25) (layer "F.Cu") (net 3))
-  (segment (start 289.44 109.22) (end 294.92 114.7) (width 0.25) (layer "F.Cu") (net 3))
-  (segment (start 241.3 109.22) (end 289.44 109.22) (width 0.25) (layer "F.Cu") (net 3))
-  (segment (start 93.004826 88.075) (end 220.155 88.075) (width 0.25) (layer "F.Cu") (net 3))
   (segment (start 51.332706 77.549509) (end 51.024418 77.549509) (width 0.25) (layer "F.Cu") (net 8))
   (segment (start 51.024418 77.549509) (end 49.59728 78.976647) (width 0.25) (layer "F.Cu") (net 8))
-  (segment (start 57.710106 63.5) (end 268.12 63.5) (width 0.25) (layer "F.Cu") (net 9))
-  (segment (start 52.74692 76.135295) (end 51.438772 76.135295) (width 0.25) (layer "F.Cu") (net 9))
-  (segment (start 48.494964 72.715142) (end 57.710106 63.5) (width 0.25) (layer "F.Cu") (net 9))
-  (segment (start 51.438772 76.135295) (end 48.494964 73.191488) (width 0.25) (layer "F.Cu") (net 9))
-  (segment (start 268.12 63.5) (end 274.32 69.7) (width 0.25) (layer "F.Cu") (net 9))
-  (segment (start 48.494964 73.191488) (end 48.494964 72.715142) (width 0.25) (layer "F.Cu") (net 9))
   (segment (start 49.092141 103.204907) (end 47.289776 101.402542) (width 0.25) (layer "F.Cu") (net 10))
   (segment (start 47.280648 101.402541) (end 47.280648 101.542541) (width 0.25) (layer "F.Cu") (net 10))
@@
   (segment (start 614.158479 110.355635) (end 614.158479 109.701211) (width 0.25) (layer "F.Cu") (net 67))
   (segment (start 614.158479 109.701211) (end 616.671128 107.188562) (width 0.25) (layer "F.Cu") (net 67))
-  (segment (start 49.63565 73.024026) (end 84.053852 73.024026) (width 0.25) (layer "F.Cu") (net 92))
-  (segment (start 84.053852 73.024026) (end 86.049791 75.019965) (width 0.25) (layer "F.Cu") (net 92))
   (segment (start 310.200035 75.019965) (end 315.52 69.7) (width 0.25) (layer "F.Cu") (net 92))
-  (segment (start 86.049791 75.019965) (end 310.200035 75.019965) (width 0.25) (layer "F.Cu") (net 92))
   (segment (start 46.13 83.825) (end 46.13 79.6868) (width 0.25) (layer "F.Cu") (net 142))
   (segment (start 46.13 79.6868) (end 46.98128 78.83552) (width 0.25) (layer "F.Cu") (net 142))

Commit message: Cap Change
Parts:
- added J2: Conn_01x02, Connector_JST:JST_XH_B2B-XH-A_1x02_P2.50mm_Vertical, F.Cu at (351.8, 80.0)
- added J3: Conn_01x02, Connector_JST:JST_XH_B2B-XH-A_1x02_P2.50mm_Vertical, F.Cu at (315.0, 82.5)
- C10, C9: footprint Capacitor_SMD:C_0603_1608Metric_Pad1.08x0.95mm_HandSolder -> Capacitor_SMD:C_0805_2012Metric_Pad1.18x1.45mm_HandSolder
- R79: footprint Resistor_SMD:R_2512_6332Metric_Pad1.40x3.35mm_HandSolder -> Resistor_SMD:R_0603_1608Metric_Pad0.98x0.95mm_HandSolder
- moved C27 527.8 mm to (633.0, 76.3), turned to -135 degrees
- moved C28 514.9 mm to (633.2, 79.5), turned to -135 degrees
- moved C38 501.7 mm to (625.9, 108.7), turned to -45 degrees
- moved C37 477.2 mm to (624.1, 102.4), turned to 0 degrees
- moved C39 456.5 mm to (628.5, 111.4), turned to -45 degrees
- moved C33 448.5 mm to (618.5, 92.1)
- moved C36 438.5 mm to (621.0, 98.4)
- moved C30 432.6 mm to (630.0, 82.6), turned to -135 degrees
- moved C29 427.8 mm to (629.9, 79.4), turned to -135 degrees
- moved C35 413.8 mm to (618.5, 96.4)
- moved C34 411.7 mm to (621.0, 94.4)
- moved C9 290.4 mm to (309.0, 78.7)
- moved C10 215.5 mm to (358.1, 82.5), turned to 0 degrees
- moved R49 51.3 mm to (39.4, 38.5)
- moved R92 51.3 mm to (44.0, 38.5)
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Connections:
- net /BatteryBus1.C13 renamed /BatteryBus1.C14
- net /C+101 renamed C+101
- net /C+102 renamed C+102
- net /C+103 renamed C+103
- net /C+104 renamed C+104
- net /C+105 renamed C+105
- net /C+106 renamed C+106
- net /C+107 renamed C+107
- net /C+108 renamed C+108
- net /C+109 renamed C+109
- net /C+110 renamed C+110
- net /C+111 renamed C+111
- net /C+112 renamed C+112
- net /C+113 renamed C+113
- net /C+201 renamed C+201
- net /C+202 renamed C+202
- net /C+203 renamed C+203
- net /C+204 renamed C+204
- net /C+205 renamed C+205
- net /C+206 renamed C+206
- net /C+207 renamed C+207
- net /C+208 renamed C+208
- net /C+209 renamed C+209
- net /C+210 renamed C+210
- net /C+211 renamed C+211
- net /C+212 renamed C+212
- net /CT101 renamed CT101
- net /CT102 renamed CT102
- net /CT103 renamed CT103
- net /CT104 renamed CT104
- net /CT105 renamed CT105
- net /CT106 renamed CT106
- net /CT107 renamed CT107
- net /CT108 renamed CT108
- net /CT109 renamed CT109
- net /CT110 renamed CT110
- net /CT111 renamed CT111
- net /CT112 renamed CT112
- net /CT113 renamed CT113
- net /CT201 renamed CT201
- net /CT202 renamed CT202
- net /CT203 renamed CT203
- net /CT204 renamed CT204
- net /CT205 renamed CT205
- net /CT206 renamed CT206
- net /CT207 renamed CT207
- net /CT208 renamed CT208
- net /CT209 renamed CT209
- net /CT210 renamed CT210
- net /CT211 renamed CT211
- net /CT212 renamed CT212
- net /D21 renamed D21
- C10 pad 1: Net-(C10-Pad1) -> Net-(J2-Pin_2)
- C15 pad 2: GND2 -> /BatteryBus1.C11
- C16 pad 2: GND2 -> /BatteryBus1.C10
- C17 pad 2: GND2 -> /BatteryBus1.C9
- C18 pad 2: GND2 -> /BatteryBus1.C8
- C19 pad 2: GND2 -> /BatteryBus1.C7
- C20 pad 2: GND2 -> /BatteryBus1.C6
- C21 pad 2: GND2 -> /BatteryBus1.C5
- C22 pad 2: GND2 -> /BatteryBus1.C4
- C23 pad 2: GND2 -> /BatteryBus1.C3
- C24 pad 2: GND2 -> /BatteryBus1.C2
- C25 pad 2: GND2 -> /BatteryBus1.C1
- C26 pad 2: GND2 -> /BatteryBus1.C0
- C27 pad 2: GND1 -> /BatteryBus.C12
- C28 pad 2: GND1 -> /BatteryBus.C11
- C29 pad 2: GND1 -> /BatteryBus.C10
- C30 pad 2: GND1 -> /BatteryBus.C9
- C31 pad 2: GND1 -> /BatteryBus.C8
- C32 pad 1: /BatteryBus.C8 -> /BatteryBus.C7
- C32 pad 2: GND1 -> /BatteryBus.C8
- C33 pad 2: GND1 -> /BatteryBus.C6
- C34 pad 2: GND1 -> /BatteryBus.C5
- C35 pad 2: GND1 -> /BatteryBus.C4
- C36 pad 2: GND1 -> /BatteryBus.C3
- C37 pad 2: GND1 -> /BatteryBus.C2
- C38 pad 2: GND1 -> /BatteryBus.C1
- C39 pad 2: GND1 -> /BatteryBus.C0
- C9 pad 2: Net-(C9-Pad2) -> Net-(J3-Pin_2)
- R3 pad 1: VDC -> VDD
- R4 pad 1: VDC -> VDD
- R7 pad 1: VDC -> VDD
- U10 pad 64: Net-(C9-Pad2) -> Net-(J2-Pin_1)
- U9 pad 61: Net-(C10-Pad1) -> Net-(J3-Pin_1)
Routing:
- net Net-(B8--): track 164.8 -> 0.00 mm, vias 1 -> 0
- net Net-(U9-C13): track 7.96 -> 0.00 mm
- net GND2: track 7.52 -> 0.00 mm
- net Net-(U9-C12): track 6.78 -> 0.00 mm
- net Net-(U9-C0): track 6.56 -> 0.00 mm
- net Net-(U9-C11): track 5.59 -> 0.00 mm
- net Net-(U9-C1): track 5.34 -> 0.00 mm
- net Net-(U9-C2): track 4.65 -> 0.00 mm
- net /BatteryBus.C1: track 4.28 -> 0.00 mm
- net /BatteryBus.C2: track 4.22 -> 0.00 mm
- net /BatteryBus.C0: track 4.21 -> 0.00 mm
- net Net-(U9-C10): track 3.99 -> 0.00 mm
- net /BatteryBus1.C10: track 3.55 -> 0.00 mm
- net /BatteryBus1.C14: track 3.10 -> 0.00 mm
- net /BatteryBus1.C11: track 3.04 -> 0.00 mm
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Other:
- board size 625.6 x 67.2 mm -> 647.7 x 67.9 mm
- rule pad_to_mask_clearance: 0 -> 0.1

Commit message: Everybody is in their general local!
Parts:
- added G***: LOGO, LOGO, F.Cu at (52.7, 28.6)
- added G***: LOGO, AERO_Footprints:AERO_Logo_25x10mm, F.Cu at (48.3, 113.7)
- moved J1 622.5 mm to (40.1, 84.7), turned to -90 degrees
- moved Q2 613.4 mm to (42.3, 37.4), turned to 0 degrees
- moved R79 601.5 mm to (44.4, 73.4)
- moved T1 599.9 mm to (51.5, 86.0), turned to 180 degrees
- moved U10 585.9 mm to (52.8, 55.6), turned to 90 degrees
- moved L23 584.5 mm to (53.3, 69.1), turned to 135 degrees
- moved L24 581.9 mm to (54.5, 67.8), turned to 135 degrees
- moved L17 580.4 mm to (55.6, 42.0), turned to -135 degrees
- moved L25 579.3 mm to (55.8, 66.5), turned to 135 degrees
- moved C28 579.0 mm to (54.2, 73.5), turned to 45 degrees
- moved L18 577.1 mm to (57.1, 43.5), turned to -135 degrees
- moved L20 576.7 mm to (57.1, 65.2), turned to 135 degrees
- moved C27 576.2 mm to (56.8, 70.8), turned to 45 degrees
- moved C39 575.6 mm to (57.5, 39.2), turned to 135 degrees
- moved L27 573.9 mm to (58.6, 45.0), turned to -135 degrees
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Connections:
- C13 pad 2: GND -> GND2
- C14 pad 2: GND -> GND1
Other:
- board size 647.7 x 67.9 mm -> 312.9 x 154.8 mm
