File: BMS1/BMS1.kicad_pcb (KiCad board)
At the start: 2 copper layers, 313 x 155.7 mm, 210 parts, among them J1 Conn_01x02, J2 Conn_01x02, J3 Conn_01x02, Q1 Q_NPN_BCE, Q2 DXT5551P5-13_DIO, T1 ESMIT-4180_C, U1 ADG728, U10 LTC6812-1, U2 ADG728, U3 ADG728, U4 ADG728, U5 ADG728, U6 ADG728, U7 ADG728, U8 ADG728, U9 LTC6812-1

Commit message: Footprints
Changed lines of the file:
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@@
 		(tags "capacitor handsolder")
 		(property "Reference" "C42"
-			(at 0 -1.43 360)
+			(at 0 -1.43 0)
 			(layer "F.SilkS")
 			(effects
@@
 		)
 		(property "Value" "1uf"
-			(at 0 1.43 360)
+			(at 0 1.43 0)
 			(layer "F.Fab")
 			(effects
@@
 		)
 		(fp_text user "${REFERENCE}"
-			(at -1.6775 1.27 360)
+			(at -1.6775 1.27 0)
 			(layer "F.Fab")
 			(effects
@@
 	)
 	(gr_text "S. Wiederman\nN. Totten\nC. Grund\nPAC BOARD v2\nB2"
-		(at 54.05 30.85 0)
+		(at 53.34 33.02 0)
 		(layer "F.SilkS")
 		(effects

Commit message: PCB
Parts:
- added C40: 1uF, Capacitor_SMD:C_0603_1608Metric, F.Cu at (120.7, 58.4)
- added Q3: DXT5551P5-13_DIO, AERO_Footprints:DXT5551P5-13_DIO, F.Cu at (318.6, 152.4)
- added R96: 100, Resistor_SMD:R_0805_2012Metric, F.Cu at (42.8, 72.4)
- added R97: 100, Resistor_SMD:R_0805_2012Metric, F.Cu at (309.9, 121.9)
- C1, C2, C3, C4, C5, C6, C7, C8: footprint Capacitor_SMD:C_0603_1608Metric_Pad1.08x0.95mm_HandSolder -> Capacitor_SMD:C_0603_1608Metric
- C10, C9: footprint Capacitor_SMD:C_0805_2012Metric_Pad1.18x1.45mm_HandSolder -> Capacitor_SMD:C_0805_2012Metric
- C11, C12, C41, C42, C43: value 1uf -> 1uF; footprint Capacitor_SMD:C_0603_1608Metric_Pad1.08x0.95mm_HandSolder -> Capacitor_SMD:C_0603_1608Metric
- C13, C14: value 100nf -> 0.1uF; footprint Capacitor_SMD:C_0603_1608Metric_Pad1.08x0.95mm_HandSolder -> Capacitor_SMD:C_0603_1608Metric
- C15, C16, C17, C18, C19, C20, C21, C22, C23, C24, C25, C26, C27, C28, C29, C30, C31, C32, C33, C34, C35, C37, C38, C39: value .1u -> 0.1uF; footprint Capacitor_SMD:C_0603_1608Metric_Pad1.08x0.95mm_HandSolder -> Capacitor_SMD:C_0603_1608Metric
- C36: value 0.1u -> 0.1uF; footprint Capacitor_SMD:C_0603_1608Metric_Pad1.08x0.95mm_HandSolder -> Capacitor_SMD:C_0603_1608Metric
- D1, D2: footprint LED_SMD:LED_0603_1608Metric_Pad1.05x0.95mm_HandSolder -> LED_SMD:LED_0201_0603Metric
- R1, R10, R11, R12, R2, R3, R39, R4, R40, R41, R42, R43, R44, R45, R46, R47, R48, R49, R5, R50, R51, R6, R7, R79, R8, R80, R81, R82, R83, R84, R85, R86, R87, R88, R89, R9, R90, R91, R92, R93, R94, R95: footprint Resistor_SMD:R_0603_1608Metric_Pad0.98x0.95mm_HandSolder -> Resistor_SMD:R_0603_1608Metric
- R13, R14, R15, R16, R17, R18, R19, R20, R21, R22, R23, R24, R25, R26, R52, R53, R55, R56, R57, R58, R59, R60, R61, R62, R63, R64, R65, R66: footprint Resistor_SMD:R_0805_2012Metric_Pad1.20x1.40mm_HandSolder -> Resistor_SMD:R_0805_2012Metric
- R27, R28, R29, R30, R31, R32, R33, R34, R35, R36, R37, R38, R67, R68, R69, R70, R71, R72, R73, R74, R75, R76, R77, R78: footprint Resistor_SMD:R_2512_6332Metric_Pad1.40x3.35mm_HandSolder -> Resistor_SMD:R_2512_6332Metric
- R54: footprint Resistor_SMD:R_0603_1608Metric_Pad0.98x0.95mm_HandSolder -> Resistor_SMD:R_0805_2012Metric
- U10, U9: footprint AERO_Footprints:LTC6812 -> AERO_Footprints:QFP-64_11x11_Pitch0.5mm
- moved C43 141.3 mm to (305.3, 120.7)
Connections:
- net /BatteryBus.C14 renamed /BatteryBus.C15
- Q2 pad 1: VCC -> Net-(Q2-B)
- Q2 pad 2: Net-(Q2-B) -> VCC
- T1 pad 1: Net-(L1-Pad3) -> /IPA
- T1 pad 2: Net-(L1-Pad2) -> /IMA
- T1 pad 3: /IPA -> Net-(L1-Pad2)
- T1 pad 4: /IMA -> Net-(L1-Pad1)
Routing:
- net (no net): track 0.00 -> 13.9 mm
- net Net-(Q3-B): track 0.00 -> 8.77 mm
- net Net-(U9-C0): track 7.70 -> 0.00 mm
- net Net-(U10-CSB(IMA)): track 32.2 -> 39.4 mm
- net Net-(U9-C1): track 6.16 -> 0.00 mm
- net CT102: track 39.9 -> 44.9 mm

Commit message: PCB Routing
Routing:
- net Net-(Q3-B): track 8.77 -> 50.7 mm
- net VDC: track 13.7 -> 46.5 mm
Changed lines of the file:
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@@
 	)
 	(segment
+		(start 322.710199 153.245001)
+		(end 322.710199 127.130199)
+		(width 0.25)
+		(layer "F.Cu")
+		(net 114)
+	)
+	(segment
+		(start 322.710199 127.130199)
+		(end 318.77 123.19)
+		(width 0.25)
+		(layer "F.Cu")
+		(net 114)
+	)
+	(segment
 		(start 314.314123 131.2348)
 		(end 313.000323 129.921)
@@
 	)
 	(segment
+		(start 322.635199 153.320001)
+		(end 322.710199 153.245001)
+		(width 0.25)
+		(layer "F.Cu")
+		(net 114)
+	)
+	(segment
 		(start 309.71 127.148499)
 		(end 309.71 129.906999)
@@
 	)
 	(segment
+		(start 321.583599 153.320001)
+		(end 322.635199 153.320001)
+		(width 0.25)
+		(layer "F.Cu")
+		(net 114)
+	)
+	(segment
 		(start 308.928001 129.971999)
 		(end 308.634 130.266)
@@
 	)
 	(segment
+		(start 317.5 152.4)
+		(end 319.440001 154.340001)
+		(width 0.25)
+		(layer "F.Cu")
+		(net 232)
+	)
+	(segment
+		(start 323.160199 126.943803)
+		(end 318.956396 122.74)
+		(width 0.25)
+		(layer "F.Cu")
+		(net 232)
+	)
+	(segment
 		(start 317.159274 152.4)
 		(end 311.201 146.441726)
@@
 	)
 	(segment
+		(start 318.32 124.01)
+		(end 318.77 124.46)
+		(width 0.25)
+		(layer "F.Cu")
+		(net 232)
+	)
+	(segment
+		(start 318.583604 122.74)
+		(end 318.32 123.003604)
+		(width 0.25)
+		(layer "F.Cu")
+		(net 232)
+	)
+	(segment
+		(start 318.32 123.003604)
+		(end 318.32 124.01)
+		(width 0.25)
+		(layer "F.Cu")
+		(net 232)
+	)
+	(segment
 		(start 317.5 152.4)
 		(end 317.159274 152.4)
 		(width 0.25)
 		(layer "F.Cu")
+		(net 232)
+	)
+	(segment
+		(start 318.956396 122.74)
+		(end 318.583604 122.74)
+		(width 0.25)
+		(layer "F.Cu")
+		(net 232)
+	)
+	(segment
+		(start 319.440001 154.340001)
+		(end 322.710199 154.340001)
+		(width 0.25)
+		(layer "F.Cu")
+		(net 232)
+	)
+	(segment
+		(start 322.710199 154.340001)
+		(end 323.160199 153.890001)
+		(width 0.25)
+		(layer "F.Cu")
+		(net 232)
+	)
+	(segment
+		(start 323.160199 153.890001)
+		(end 323.160199 126.943803)
+		(width 0.25)
+		(layer "F.Cu")
