File: BMS1/BMS1.kicad_pcb (KiCad board)
At the start: 2 copper layers, 313 x 155.7 mm, 214 parts, among them J1 Conn_01x02, J2 Conn_01x02, J3 Conn_01x02, Q1 Q_NPN_BCE, Q2 DXT5551P5-13_DIO, Q3 DXT5551P5-13_DIO, T1 ESMIT-4180_C, U1 ADG728, U10 LTC6812-1, U2 ADG728, U3 ADG728, U4 ADG728, U5 ADG728, U6 ADG728, U7 ADG728, U8 ADG728, U9 LTC6812-1

Commit message: PCB Routing
Routing:
- net VDD: track 368.1 -> 375.4 mm, vias 5 -> 7
- net Net-(U9-SCK(IPA)): track 20.8 -> 23.3 mm
- net GND2: vias 68 -> 69
Changed lines of the file:
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@@
+	)
+	(segment
+		(start 321.583599 148.863599)
+		(end 321.31 148.59)
+		(width 0.25)
+		(layer "F.Cu")
+		(net 75)
 	)
 	(segment
@@
 	)
 	(segment
+		(start 321.583599 151.479999)
+		(end 321.583599 148.863599)
+		(width 0.25)
+		(layer "F.Cu")
+		(net 75)
+	)
+	(segment
 		(start 188.4635 150.267)
 		(end 190.378501 150.267)
@@
 		(net 75)
 	)
+	(via
+		(at 320.04 144.78)
+		(size 0.8)
+		(drill 0.4)
+		(layers "F.Cu" "B.Cu")
+		(free yes)
+		(net 75)
+	)
+	(via
+		(at 321.31 148.59)
+		(size 0.8)
+		(drill 0.4)
+		(layers "F.Cu" "B.Cu")
+		(free yes)
+		(net 75)
+	)
+	(segment
+		(start 321.31 146.05)
+		(end 320.04 144.78)
+		(width 0.25)
+		(layer "B.Cu")
+		(net 75)
+	)
 	(segment
 		(start 210.884 130.556)
 		(end 212.154 129.286)
+		(width 0.25)
+		(layer "B.Cu")
+		(net 75)
+	)
+	(segment
+		(start 321.31 148.59)
+		(end 321.31 146.05)
 		(width 0.25)
 		(layer "B.Cu")
@@
 	)
 	(via
+		(at 312.42 119.38)
+		(size 0.8)
+		(drill 0.4)
+		(layers "F.Cu" "B.Cu")
+		(free yes)
+		(net 76)
+	)
+	(via
 		(at 238.824 141.859)
 		(size 0.8)
@@
 	)
 	(segment
+		(start 310.7925 121.0075)
+		(end 311.907348 119.892652)
+		(width 0.25)
+		(layer "F.Cu")
+		(net 85)
+	)
+	(segment
 		(start 315.913 121.158)
 		(end 315.913 119.677)
@@
 		(width 0.25)
 		(layer "F.Cu")
+		(net 85)
+	)
+	(segment
+		(start 309.88 121.0075)
+		(end 310.7925 121.0075)
+		(width 0.25)
+		(layer "F.Cu")

Commit message: Routing
Parts:
- moved L1 252.4 mm to (61.0, 80.0), turned to -45 degrees
- moved C40 71.6 mm to (51.4, 40.4), turned to 180 degrees
- moved C42 14.8 mm to (149.1, 59.7)
- moved C9 9.11 mm to (307.3, 115.6)
- moved T1 4.58 mm to (51.3, 86.9), turned to -90 degrees
- moved R97 2.84 mm to (312.4, 120.7)
- moved C43 1.61 mm to (304.3, 121.9)
- moved L2 0.52 mm to (304.8, 152.4), turned to -135 degrees
Routing:
- net GND1: track 54.2 -> 176.9 mm, vias 46 -> 54
- net GND2: track 311.8 -> 425.0 mm, vias 69 -> 70
- net Net-(B7-+): track 151.3 -> 174.8 mm
- net Net-(B9-+): track 187.0 -> 210.5 mm
- net Net-(B11-+): track 229.4 -> 252.9 mm
- net Net-(B5-+): track 114.9 -> 138.2 mm
- net Net-(B8-+): track 164.2 -> 185.1 mm, vias 1 -> 2
- net Net-(B3-+): track 71.5 -> 92.3 mm
- net Net-(B6-+): track 115.1 -> 135.9 mm
- net Net-(B16-+): track 302.9 -> 323.6 mm
- net Net-(B12-+): track 310.2 -> 330.8 mm
- net Net-(B22-+): track 88.0 -> 108.6 mm
- net Net-(B20-+): track 131.5 -> 152.1 mm
- net Net-(B4-+): track 63.1 -> 83.7 mm
- net Net-(B10-+): track 246.0 -> 266.6 mm
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
Commit message: MOre Routinggggg
Parts:
- removed the G*** at (309.1, 169.4)
- removed L10, L11, L12, L13, L14, L15, L16, L17, L18, L20, L21, L23, L24, L25, L26, L27, L28, L29, L3, L30, L31, L32, L4, L7, L8, L9: L_Ferrite_Small, Inductor_SMD:L_0603_1608Metric_Pad1.05x0.95mm_HandSolder
- removed Q1: Q_NPN_BCE, AERO_Footprints:DXT5551P5-13_DIO
- B1, B4: moved to B.Cu
- moved C41 39.5 mm to (320.0, 141.7), turned to 90 degrees
- moved L2 37.0 mm to (308.6, 115.6), turned to 135 degrees
- moved C43 8.11 mm to (311.1, 126.3), turned to 90 degrees
- moved C9 2.84 mm to (304.8, 114.3)
- moved R3 2.09 mm to (307.8, 152.4)
- turned B1 to 0 degrees
- turned B4 to 180 degrees
Connections:
- net /BatteryBus.C15 renamed /BatteryBus.C14
- T1 pad 3: Net-(L1-Pad2) -> Net-(L1-Pad3)
- T1 pad 4: Net-(L1-Pad1) -> Net-(L1-Pad2)
Routing:
- net Net-(U9-CSB(IMA)): track 0.00 -> 60.5 mm, vias 0 -> 2
- net Net-(U9-VREF2): track 0.00 -> 35.2 mm, vias 0 -> 2
- net Net-(Q1-B): track 32.8 -> 0.00 mm
- net /BatteryBus1.C13: track 0.00 -> 29.3 mm
- net Net-(U10-ICMP): track 6.60 -> 35.3 mm, vias 0 -> 3
- net /BatteryBus1.C14: track 19.1 -> 0.00 mm
- net Net-(U10-CSB(IMA)): track 37.5 -> 56.1 mm, vias 2 -> 3
- net Net-(B25-+): track 61.1 -> 77.4 mm
- net Net-(L1-Pad3): track 0.00 -> 16.2 mm
- net VDC: track 59.8 -> 47.7 mm
- net Net-(J3-Pin_1): track 32.7 -> 43.4 mm, vias 2 -> 1
- net GND2: track 425.0 -> 414.6 mm
- net /BatteryBus1.C3: track 9.91 -> 20.3 mm
- net /BatteryBus.C0: track 5.48 -> 15.5 mm
- net /BatteryBus1.C12: track 5.62 -> 15.5 mm
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