File: BMS1/Section1.kicad_sch (KiCad schematic)
At the start: 68 parts

Commit message: Meeting 11/14/24
Connections:
- net at B23.1 (+), R61.1, R77.1: no longer B22.2 (-)
- net at B18.1 (+), R63.1, R74.1: no longer B17.2 (-)
- net at B22.1 (+), R52.1, R68.1: no longer B21.2 (-)
- net at B25.1 (+), R53.1, R69.1: no longer B24.2 (-)
- net at B19.1 (+), R64.1, R76.1: no longer B18.2 (-)
- net at B20.1 (+), R65.1, R78.1: no longer B19.2 (-)
- net at B17.1 (+), R62.1, R73.1: no longer B16.2 (-)
- net at B21.1 (+), R60.1, R71.1: no longer B20.2 (-)
- net at B16.1 (+), R56.1, R70.1: no longer B15.2 (-)
- net at B14.1 (+), R59.1, R72.1: no longer B13.2 (-)
- net at B15.1 (+), R55.1, R67.1: no longer B14.2 (-)
Changed lines of the file:
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@@
   (junction (at 99.314 34.417) (diameter 0) (color 0 0 0 0)
   )
-  (junction (at 80.391 166.624) (diameter 0) (color 0 0 0 0)
-  )
   (junction (at 79.375 34.417) (diameter 0) (color 0 0 0 0)
   )
   (junction (at 69.215 34.417) (diameter 0) (color 0 0 0 0)
   )
-  (junction (at 80.391 75.184) (diameter 0) (color 0 0 0 0)
-  )
   (junction (at 99.314 141.224) (diameter 0) (color 0 0 0 0)
   )
@@
   (junction (at 40.259 115.824) (diameter 0) (color 0 0 0 0)
   )
-  (junction (at 80.391 151.384) (diameter 0) (color 0 0 0 0)
-  )
   (junction (at 80.391 95.504) (diameter 0) (color 0 0 0 0)
   )
@@
   (junction (at 40.259 161.544) (diameter 0) (color 0 0 0 0)
   )
-  (junction (at 80.518 212.344) (diameter 0) (color 0 0 0 0)
-  )
   (junction (at 66.294 227.584) (diameter 0) (color 0 0 0 0)
   )
-  (junction (at 80.391 44.577) (diameter 0) (color 0 0 0 0)
-  )
   (junction (at 80.391 156.464) (diameter 0) (color 0 0 0 0)
   )
-  (junction (at 80.391 120.904) (diameter 0) (color 0 0 0 0)
-  )
   (junction (at 99.314 65.024) (diameter 0) (color 0 0 0 0)
   )
@@
   (junction (at 40.259 222.504) (diameter 0) (color 0 0 0 0)
   )
-  (junction (at 80.391 181.864) (diameter 0) (color 0 0 0 0)
-  )
   (junction (at 99.314 227.584) (diameter 0) (color 0 0 0 0)
   )
@@
   (junction (at 80.391 125.984) (diameter 0) (color 0 0 0 0)
   )
-  (junction (at 80.391 105.664) (diameter 0) (color 0 0 0 0)
-  )
-  (junction (at 80.391 59.944) (diameter 0) (color 0 0 0 0)
-  )
   (junction (at 99.314 217.424) (diameter 0) (color 0 0 0 0)
   )
@@
   )
   (junction (at 80.391 202.184) (diameter 0) (color 0 0 0 0)
-  )
-  (junction (at 80.391 90.424) (diameter 0) (color 0 0 0 0)
-  )
-  (junction (at 80.391 136.144) (diameter 0) (color 0 0 0 0)
   )
   (junction (at 99.314 95.504) (diameter 0) (color 0 0 0 0)
@@
     (stroke (width 0) (type default))
   )
-  (wire (pts (xy 80.391 181.864) (xy 65.024 181.864))
-    (stroke (width 0) (type default))
-  )
   (wire (pts (xy 40.259 32.893) (xy 40.259 39.497))
     (stroke (width 0) (type default))
@@
     (stroke (width 0) (type default))
   )
-  (wire (pts (xy 80.391 151.384) (xy 65.024 151.384))
-    (stroke (width 0) (type default))
-  )
   (wire (pts (xy 116.586 44.577) (xy 90.043 44.577))
     (stroke (width 0) (type default))
@@
     (stroke (width 0) (type default))
   )
-  (wire (pts (xy 80.518 212.344) (xy 65.024 212.344))
-    (stroke (width 0) (type default))
-  )
   (wire (pts (xy 25.019 176.784) (xy 32.385 176.784))
     (stroke (width 0) (type default))
@@
     (stroke (width 0) (type default))
   )
-  (wire (pts (xy 65.024 75.184) (xy 80.391 75.184))
-    (stroke (width 0) (type default))
-  )
   (wire (pts (xy 40.259 215.9) (xy 40.259 222.504))
     (stroke (width 0) (type default))
@@
     (stroke (width 0) (type default))
   )
-  (wire (pts (xy 65.024 44.577) (xy 80.391 44.577))
-    (stroke (width 0) (type default))
-  )
   (wire (pts (xy 98.298 217.424) (xy 99.314 217.424))
     (stroke (width 0) (type default))
@@
     (stroke (width 0) (type default))
   )
-  (wire (pts (xy 80.391 120.904) (xy 65.024 120.904))
-    (stroke (width 0) (type default))
-  )
   (wire (pts (xy 99.314 49.784) (xy 116.586 49.784))
     (stroke (width 0) (type default))
@@
     (stroke (width 0) (type default))
   )
-  (wire (pts (xy 80.391 166.624) (xy 65.024 166.624))
-    (stroke (width 0) (type default))
-  )
   (wire (pts (xy 90.297 75.184) (xy 116.586 75.184))
     (stroke (width 0) (type default))
@@
     (stroke (width 0) (type default))
   )
-  (wire (pts (xy 80.391 90.424) (xy 65.024 90.424))
-    (stroke (width 0) (type default))
-  )
   (bus (pts (xy 119.126 35.306) (xy 119.126 32.131))
     (stroke (width 0) (type default))
@@
     (stroke (width 0) (type default))
   )
-  (wire (pts (xy 80.391 136.144) (xy 65.024 136.144))
-    (stroke (width 0) (type default))
-  )
   (wire (pts (xy 99.314 95.504) (xy 99.314 97.282))
     (stroke (width 0) (type default))
@@
     (stroke (width 0) (type default))
   )
-  (wire (pts (xy 80.391 59.944) (xy 65.024 59.944))
-    (stroke (width 0) (type default))
-  )
   (wire (pts (xy 40.259 115.824) (xy 47.244 115.824))
     (stroke (width 0) (type default))
@@
     (stroke (width 0) (type default))
   )
-  (wire (pts (xy 80.391 105.664) (xy 65.024 105.664))
-    (stroke (width 0) (type default))
-  )
