File: BMS1/Section1.kicad_sch (KiCad schematic)
At the start: 68 parts

Commit message: updated datasheets and MPNs
Parts:
- R67, R68, R69, R70, R71, R72, R73, R74, R75, R76, R77, R78, R79: MPN (none) -> RMCF2512FT18R0
Changed lines of the file:
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@@
 			)
 		)
-		(property "Datasheet" "~"
+		(property "Datasheet" "https://www.seielect.com/catalog/sei-rmcf_rmcp.pdf"
 			(at 85.09 182.88 0)
 			(effects
@@
 			)
 		)
-		(property "MPN" ""
+		(property "MPN" "RMCF2512FT18R0"
 			(at 85.09 182.88 0)
 			(effects
@@
 			)
 		)
-		(property "Datasheet" "~"
+		(property "Datasheet" "https://www.seielect.com/catalog/sei-rmcf_rmcp.pdf"
 			(at 85.09 106.68 0)
 			(effects
@@
 			)
 		)
-		(property "MPN" ""
+		(property "MPN" "RMCF2512FT18R0"
 			(at 85.09 106.68 0)
 			(effects
@@
 			)
 		)
-		(property "Datasheet" "~"
+		(property "Datasheet" "https://www.seielect.com/catalog/sei-rmcf_rmcp.pdf"
 			(at 87.63 167.64 0)
 			(effects
@@
 			)
 		)
-		(property "MPN" ""
+		(property "MPN" "RMCF2512FT18R0"
 			(at 87.63 167.64 0)
 			(effects
@@
 			)
 		)
-		(property "Datasheet" "~"
+		(property "Datasheet" "https://www.seielect.com/catalog/sei-rmcf_rmcp.pdf"
 			(at 87.63 213.36 0)
 			(effects
@@
 			)
 		)
-		(property "MPN" ""
+		(property "MPN" "RMCF2512FT18R0"
 			(at 87.63 213.36 0)
 			(effects
@@
 			)
 		)
-		(property "Datasheet" "~"
+		(property "Datasheet" "https://www.seielect.com/catalog/sei-rmcf_rmcp.pdf"
 			(at 85.09 121.92 0)
 			(effects
@@
 			)
 		)
-		(property "MPN" ""
+		(property "MPN" "RMCF2512FT18R0"
 			(at 85.09 121.92 0)
 			(effects
@@
 			)
 		)
-		(property "Datasheet" "~"
+		(property "Datasheet" "https://www.seielect.com/catalog/sei-rmcf_rmcp.pdf"
 			(at 85.09 30.48 0)
 			(effects
@@
 			)
 		)
-		(property "MPN" ""
+		(property "MPN" "RMCF2512FT18R0"
 			(at 85.09 30.48 0)
 			(effects
@@
 			)
 		)
-		(property "Datasheet" "~"
+		(property "Datasheet" "https://www.seielect.com/catalog/sei-rmcf_rmcp.pdf"
 			(at 85.09 91.44 0)
 			(effects
@@
 			)
 		)
-		(property "MPN" ""
+		(property "MPN" "RMCF2512FT18R0"
 			(at 85.09 91.44 0)
 			(effects
@@
 			)
 		)
-		(property "Datasheet" "~"
+		(property "Datasheet" "https://www.seielect.com/catalog/sei-rmcf_rmcp.pdf"
 			(at 87.63 152.4 0)
 			(effects
@@
 			)
 		)
-		(property "MPN" ""
+		(property "MPN" "RMCF2512FT18R0"
 			(at 87.63 152.4 0)
 			(effects
@@
 			)
 		)
-		(property "Datasheet" "~"
+		(property "Datasheet" "https://www.seielect.com/catalog/sei-rmcf_rmcp.pdf"
 			(at 85.09 45.72 0)
 			(effects
@@
 			)
 		)
-		(property "MPN" ""
+		(property "MPN" "RMCF2512FT18R0"
 			(at 85.09 45.72 0)
 			(effects
@@
 			)
 		)
-		(property "Datasheet" "~"
+		(property "Datasheet" "https://www.seielect.com/catalog/sei-rmcf_rmcp.pdf"
 			(at 85.09 198.12 0)
 			(effects
@@
 			)
 		)
-		(property "MPN" ""
+		(property "MPN" "RMCF2512FT18R0"
 			(at 85.09 198.12 0)
 			(effects
@@
 			)
 		)
-		(property "Datasheet" "~"
+		(property "Datasheet" "https://www.seielect.com/catalog/sei-rmcf_rmcp.pdf"
 			(at 87.63 60.96 0)
 			(effects
@@
 			)
 		)
-		(property "MPN" ""
+		(property "MPN" "RMCF2512FT18R0"
 			(at 87.63 60.96 0)
 			(effects
@@
 			)
 		)
-		(property "Datasheet" "~"
+		(property "Datasheet" "https://www.seielect.com/catalog/sei-rmcf_rmcp.pdf"
 			(at 85.09 137.16 0)
 			(effects
@@
 			)
 		)
-		(property "MPN" ""
+		(property "MPN" "RMCF2512FT18R0"
 			(at 85.09 137.16 0)
 			(effects
@@
 			)
 		)
-		(property "Datasheet" "~"
+		(property "Datasheet" "https://www.seielect.com/catalog/sei-rmcf_rmcp.pdf"
 			(at 87.63 76.2 0)
 			(effects
@@
 			)
 		)
-		(property "MPN" ""
+		(property "MPN" "RMCF2512FT18R0"
 			(at 87.63 76.2 0)
 			(effects

Commit message: DRC error fixes
Parts:
- C27, C28, C29, C30, C31, C32, C33, C34, C35, C36, C37, C38, C39: Digikey Part Number (none) -> 1276-6807-1-ND; MPN AGC0603X7R101-104KXP -> CL10B104KC8NNNC
- R52, R53, R55, R56, R57, R58, R59, R60, R61, R62, R63, R64, R65, R66: Digikey Part Number (none) -> P10ADCT-ND
- R54, R80: Digikey Part Number (none) -> RMCF0805FT100RCT-ND
- R67, R68, R69, R70, R71, R72, R73, R74, R75, R76, R77, R78, R79: Digikey Part Number (none) -> RMCF2512FT18R0CT-ND
- R81, R82, R83, R84, R85, R86, R87, R88, R89, R90, R91, R92, R93: Digikey Part Number (none) -> 311-680GRCT-ND

Commit message: BOM updates
Parts:
- R79: footprint Resistor_SMD:R_0603_1608Metric -> Resistor_SMD:R_2512_6332Metric
- R80: Digikey Part Number RMCF0805FT100RCT-ND -> 311-100HRCT-ND; MPN ERJ-3EKF1000V -> RC0603FR-07100RL
Changed lines of the file:
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@@
 			)
 		)
-		(property "Footprint" "Resistor_SMD:R_0603_1608Metric"
+		(property "Footprint" "Resistor_SMD:R_2512_6332Metric"
 			(at 85.344 31.496 90)
 			(effects
@@
 			)
 		)
-		(property "Datasheet" "https://industrial.panasonic.com/cdbs/www-data/pdf/RDA0000/AOA0000C304.pdf"
+		(property "Datasheet" "https://www.yageo.com/upload/media/product/products/datasheet/rchip/PYu-RC_Group_51_RoHS_L_12.pdf"
 			(at 68.58 29.21 0)
 			(effects
@@
 			)
 		)
-		(property "MPN" "ERJ-3EKF1000V"
+		(property "MPN" "RC0603FR-07100RL"
 			(at 68.58 29.21 0)
 			(effects
@@
 			)
 		)
-		(property "Digikey Part Number" "RMCF0805FT100RCT-ND"
+		(property "Digikey Part Number" "311-100HRCT-ND"
 			(at 68.58 29.21 0)
 			(effects
