File: BMS1/Section2.kicad_sch (KiCad schematic)
At the start: 63 parts

Commit message: Cap Change
Connections:
- net BatteryBus1.C0: now also C26.2
- net BatteryBus1.C1: now also C25.2
- net BatteryBus1.C10: now also C16.2
- net BatteryBus1.C11: now also C15.2
- net BatteryBus1.C2: now also C24.2
- net BatteryBus1.C3: now also C23.2
- net BatteryBus1.C4: now also C22.2
- net BatteryBus1.C5: now also C21.2
- net BatteryBus1.C6: now also C20.2
- net BatteryBus1.C7: now also C19.2
- net BatteryBus1.C8: now also C18.2
- net BatteryBus1.C9: now also C17.2
- net GND2: no longer C15.2, C16.2, C17.2, C18.2, C19.2, C20.2, C21.2, C22.2, C23.2, C24.2, C25.2, C26.2
Other:
- moved on the sheet: C15, C16, C17, C18, C19, C20, C21, C22, C23, C24, C25, C26

Commit message: Schematic (Self) Review Done
Parts:
- C15, C16, C17, C18, C19, C20, C21, C22, C23, C24, C25, C26: value 100nF -> 15u
- R27, R28, R29, R30, R31, R32, R33, R34, R35, R36, R37, R38: value 21 -> 18
Changed lines of the file:
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@@
       (effects (font (size 1.27 1.27)) (justify right))
     )
-    (property "Value" "21" (at 99.695 100.33 90)
+    (property "Value" "18" (at 99.695 100.33 90)
       (effects (font (size 1.27 1.27)) (justify right))
     )
@@
       (effects (font (size 1.27 1.27)) (justify right))
     )
-    (property "Value" "21" (at 99.949 39.751 90)
+    (property "Value" "18" (at 99.949 39.751 90)
       (effects (font (size 1.27 1.27)) (justify right))
     )
@@
       (effects (font (size 1.27 1.27)) (justify right))
     )
-    (property "Value" "21" (at 101.727 54.483 90)
+    (property "Value" "18" (at 101.727 54.483 90)
       (effects (font (size 1.27 1.27)) (justify right))
     )
@@
       (effects (font (size 1.27 1.27)))
     )
-    (property "Value" "100nF" (at 117.856 91.186 0)
+    (property "Value" "15u" (at 117.856 91.186 0)
       (effects (font (size 1.27 1.27)))
     )
@@
       (effects (font (size 1.27 1.27)) (justify right))
     )
-    (property "Value" "21" (at 99.06 130.81 90)
+    (property "Value" "18" (at 99.06 130.81 90)
       (effects (font (size 1.27 1.27)) (justify right))
     )
@@
       (effects (font (size 1.27 1.27)))
     )
-    (property "Value" "100nF" (at 117.856 212.344 0)
+    (property "Value" "15u" (at 117.856 212.344 0)
       (effects (font (size 1.27 1.27)))
     )
@@
       (effects (font (size 1.27 1.27)))
     )
-    (property "Value" "100nF" (at 117.602 121.666 0)
+    (property "Value" "15u" (at 117.602 121.666 0)
       (effects (font (size 1.27 1.27)))
     )
@@
       (effects (font (size 1.27 1.27)))
     )
-    (property "Value" "100nF" (at 117.856 166.878 0)
+    (property "Value" "15u" (at 117.856 166.878 0)
       (effects (font (size 1.27 1.27)))
     )
@@
       (effects (font (size 1.27 1.27)))
     )
-    (property "Value" "100nF" (at 117.602 75.946 0)
+    (property "Value" "15u" (at 117.602 75.946 0)
       (effects (font (size 1.27 1.27)))
     )
@@
       (effects (font (size 1.27 1.27)) (justify right))
     )
-    (property "Value" "21" (at 100.203 161.163 90)
+    (property "Value" "18" (at 100.203 161.163 90)
       (effects (font (size 1.27 1.27)) (justify right))
     )
@@
       (effects (font (size 1.27 1.27)))
     )
-    (property "Value" "100nF" (at 117.856 151.638 0)
+    (property "Value" "15u" (at 117.856 151.638 0)
       (effects (font (size 1.27 1.27)))
     )
@@
       (effects (font (size 1.27 1.27)))
     )
-    (property "Value" "100nF" (at 117.602 182.372 0)
+    (property "Value" "15u" (at 117.602 182.372 0)
       (effects (font (size 1.27 1.27)))
     )
@@
       (effects (font (size 1.27 1.27)))
     )
-    (property "Value" "100nF" (at 117.856 197.612 0)
+    (property "Value" "15u" (at 117.856 197.612 0)
       (effects (font (size 1.27 1.27)))
     )
@@
       (effects (font (size 1.27 1.27)))
     )
-    (property "Value" "100nF" (at 117.856 136.906 0)
+    (property "Value" "15u" (at 117.856 136.906 0)
       (effects (font (size 1.27 1.27)))
     )
@@
       (effects (font (size 1.27 1.27)) (justify right))
     )
-    (property "Value" "21" (at 99.568 85.344 90)
+    (property "Value" "18" (at 99.568 85.344 90)
       (effects (font (size 1.27 1.27)) (justify right))
     )
@@
       (effects (font (size 1.27 1.27)) (justify right))
     )
-    (property "Value" "21" (at 99.949 145.796 90)
+    (property "Value" "18" (at 99.949 145.796 90)
       (effects (font (size 1.27 1.27)) (justify right))
     )
@@
       (effects (font (size 1.27 1.27)) (justify right))
     )
-    (property "Value" "21" (at 99.314 176.53 90)
+    (property "Value" "18" (at 99.314 176.53 90)
       (effects (font (size 1.27 1.27)) (justify right))
     )
@@
       (effects (font (size 1.27 1.27)) (justify right))
     )
-    (property "Value" "21" (at 99.949 70.104 90)
+    (property "Value" "18" (at 99.949 70.104 90)
       (effects (font (size 1.27 1.27)) (justify right))
     )
@@
       (effects (font (size 1.27 1.27)) (justify right))
     )
-    (property "Value" "21" (at 99.695 115.697 90)
+    (property "Value" "18" (at 99.695 115.697 90)
       (effects (font (size 1.27 1.27)) (justify right))
     )
@@
       (effects (font (size 1.27 1.27)))
     )
-    (property "Value" "100nF" (at 117.602 45.466 0)
+    (property "Value" "15u" (at 117.602 45.466 0)
       (effects (font (size 1.27 1.27)))
     )
@@
       (effects (font (size 1.27 1.27)) (justify right))
     )
-    (property "Value" "21" (at 99.695 191.77 90)
+    (property "Value" "18" (at 99.695 191.77 90)
       (effects (font (size 1.27 1.27)) (justify right))
     )
@@
       (effects (font (size 1.27 1.27)))
     )
-    (property "Value" "100nF" (at 117.602 60.198 0)
+    (property "Value" "15u" (at 117.602 60.198 0)
       (effects (font (size 1.27 1.27)))
     )
@@
       (effects (font (size 1.27 1.27)) (justify right))
     )
-    (property "Value" "21" (at 100.457 206.883 90)
+    (property "Value" "18" (at 100.457 206.883 90)
       (effects (font (size 1.27 1.27)) (justify right))
     )
@@
       (effects (font (size 1.27 1.27)))
     )
-    (property "Value" "100nF" (at 117.602 106.172 0)
-      (effects (font (size 1.27 1.27)))
-    )
+    (property "Value" "15u" (at 117.602 106.172 0)
+      (effects (font (size 1.27 1.27)))
+    )

Commit message: fixed to whats on board footy not changed
Parts:
- C15, C16, C17, C18, C19, C20, C21, C22, C23, C24, C25, C26: value 15u -> .1u
Changed lines of the file:
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@@
       (effects (font (size 1.27 1.27)))
     )
-    (property "Value" "15u" (at 117.856 91.186 0)
+    (property "Value" ".1u" (at 117.856 91.186 0)
       (effects (font (size 1.27 1.27)))
     )
@@
       (effects (font (size 1.27 1.27)))
     )
-    (property "Value" "15u" (at 117.856 212.344 0)
+    (property "Value" ".1u" (at 117.856 212.344 0)
       (effects (font (size 1.27 1.27)))
     )
@@
       (effects (font (size 1.27 1.27)))
     )
-    (property "Value" "15u" (at 117.602 121.666 0)
+    (property "Value" ".1u" (at 117.602 121.666 0)
       (effects (font (size 1.27 1.27)))
     )
@@
       (effects (font (size 1.27 1.27)))
     )
-    (property "Value" "15u" (at 117.856 166.878 0)
+    (property "Value" ".1u" (at 117.856 166.878 0)
       (effects (font (size 1.27 1.27)))
     )
@@
       (effects (font (size 1.27 1.27)))
     )
-    (property "Value" "15u" (at 117.602 75.946 0)
+    (property "Value" ".1u" (at 117.602 75.946 0)
       (effects (font (size 1.27 1.27)))
     )
@@
       (effects (font (size 1.27 1.27)))
     )
-    (property "Value" "15u" (at 117.856 151.638 0)
+    (property "Value" ".1u" (at 117.856 151.638 0)
       (effects (font (size 1.27 1.27)))
     )
@@
       (effects (font (size 1.27 1.27)))
     )
-    (property "Value" "15u" (at 117.602 182.372 0)
+    (property "Value" ".1u" (at 117.602 182.372 0)
       (effects (font (size 1.27 1.27)))
     )
@@
       (effects (font (size 1.27 1.27)))
     )
-    (property "Value" "15u" (at 117.856 197.612 0)
+    (property "Value" ".1u" (at 117.856 197.612 0)
       (effects (font (size 1.27 1.27)))
     )
@@
       (effects (font (size 1.27 1.27)))
     )
-    (property "Value" "15u" (at 117.856 136.906 0)
+    (property "Value" ".1u" (at 117.856 136.906 0)
       (effects (font (size 1.27 1.27)))
     )
@@
       (effects (font (size 1.27 1.27)))
     )
-    (property "Value" "15u" (at 117.602 45.466 0)
+    (property "Value" ".1u" (at 117.602 45.466 0)
       (effects (font (size 1.27 1.27)))
     )
@@
       (effects (font (size 1.27 1.27)))
     )
-    (property "Value" "15u" (at 117.602 60.198 0)
+    (property "Value" ".1u" (at 117.602 60.198 0)
       (effects (font (size 1.27 1.27)))
     )
@@
       (effects (font (size 1.27 1.27)))
     )
-    (property "Value" "15u" (at 117.602 106.172 0)
-      (effects (font (size 1.27 1.27)))
-    )
+    (property "Value" ".1u" (at 117.602 106.172 0)
+      (effects (font (size 1.27 1.27)))
+    )

Commit message: Meeting 11/14/24
Connections:
- net at B8.1 (+), R21.1, R31.1: no longer B7.2 (-)
- net at B9.1 (+), R15.1, R28.1: no longer B8.2 (-)
- net at B10.1 (+), R22.1, R37.1: no longer B9.2 (-)
- net at B12.1 (+), R16.1, R29.1: no longer B11.2 (-)
- net at B7.1 (+), R26.1, R38.1: no longer B6.2 (-)
- net at B11.1 (+), R19.1, R35.1: no longer B10.2 (-)
Changed lines of the file:
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@@
   (junction (at 57.658 47.244) (diameter 0) (color 0 0 0 0)
   )
-  (junction (at 95.123 174.244) (diameter 0) (color 0 0 0 0)
-  )
   (junction (at 134.874 124.46) (diameter 0) (color 0 0 0 0)
   )
@@
   (junction (at 114.554 87.884) (diameter 0) (color 0 0 0 0)
   )
-  (junction (at 95.123 128.524) (diameter 0) (color 0 0 0 0)
-  )
   (junction (at 95.123 87.884) (diameter 0) (color 0 0 0 0)
   )
-  (junction (at 95.123 159.004) (diameter 0) (color 0 0 0 0)
-  )
   (junction (at 58.166 174.244) (diameter 0) (color 0 0 0 0)
   )
@@
   (junction (at 95.123 52.324) (diameter 0) (color 0 0 0 0)
   )
-  (junction (at 95.123 189.484) (diameter 0) (color 0 0 0 0)
-  )
   (junction (at 114.554 57.404) (diameter 0) (color 0 0 0 0)
   )
   (junction (at 160.528 58.547) (diameter 0) (color 0 0 0 0)
   )
-  (junction (at 95.25 204.724) (diameter 0) (color 0 0 0 0)
-  )
   (junction (at 114.554 118.364) (diameter 0) (color 0 0 0 0)
   )
@@
   )
   (junction (at 55.372 77.724) (diameter 0) (color 0 0 0 0)
-  )
-  (junction (at 95.123 143.764) (diameter 0) (color 0 0 0 0)
   )
   (no_connect (at 158.496 53.594))
@@
     (stroke (width 0) (type default))
   )
-  (wire (pts (xy 95.25 204.724) (xy 79.756 204.724))
-    (stroke (width 0) (type default))
-  )
   (wire (pts (xy 114.554 133.604) (xy 114.554 135.382))
     (stroke (width 0) (type default))
@@
     (stroke (width 0) (type default))
   )
-  (wire (pts (xy 95.123 159.004) (xy 79.756 159.004))
-    (stroke (width 0) (type default))
-  )
   (wire (pts (xy 114.554 57.404) (xy 132.334 57.404))
     (stroke (width 0) (type default))
@@
     (stroke (width 0) (type default))
   )
-  (wire (pts (xy 95.123 128.524) (xy 79.756 128.524))
-    (stroke (width 0) (type default))
-  )
   (wire (pts (xy 112.014 133.604) (xy 114.554 133.604))
     (stroke (width 0) (type default))
@@
     (stroke (width 0) (type default))
   )
-  (wire (pts (xy 95.123 189.484) (xy 79.756 189.484))
-    (stroke (width 0) (type default))
-  )
   (wire (pts (xy 55.245 77.724) (xy 55.372 77.724))
     (stroke (width 0) (type default))
@@
     (stroke (width 0) (type default))
   )
-  (wire (pts (xy 95.123 143.764) (xy 79.756 143.764))
-    (stroke (width 0) (type default))
-  )
   (wire (pts (xy 112.649 87.884) (xy 114.554 87.884))
     (stroke (width 0) (type default))
@@
     (stroke (width 0) (type default))
   )
-  (wire (pts (xy 95.123 174.244) (xy 79.756 174.244))
-    (stroke (width 0) (type default))
-  )
