File: BMS1/Section2.kicad_sch (KiCad schematic)
At the start: 63 parts

Commit message: updated datasheets and MPNs
Parts:
- R27, R28, R29, R30, R31, R32, R33, R34, R35, R36, R37, R38: MPN (none) -> RMCF2512FT18R0
Changed lines of the file:
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@@
 			)
 		)
-		(property "Datasheet" "~"
+		(property "Datasheet" "https://www.seielect.com/catalog/sei-rmcf_rmcp.pdf"
 			(at 100.33 99.06 0)
 			(effects
@@
 			)
 		)
-		(property "MPN" ""
+		(property "MPN" "RMCF2512FT18R0"
 			(at 100.33 99.06 0)
 			(effects
@@
 			)
 		)
-		(property "Datasheet" "~"
+		(property "Datasheet" "https://www.seielect.com/catalog/sei-rmcf_rmcp.pdf"
 			(at 100.33 38.1 0)
 			(effects
@@
 			)
 		)
-		(property "MPN" ""
+		(property "MPN" "RMCF2512FT18R0"
 			(at 100.33 38.1 0)
 			(effects
@@
 			)
 		)
-		(property "Datasheet" "~"
+		(property "Datasheet" "https://www.seielect.com/catalog/sei-rmcf_rmcp.pdf"
 			(at 102.87 53.34 0)
 			(effects
@@
 			)
 		)
-		(property "MPN" ""
+		(property "MPN" "RMCF2512FT18R0"
 			(at 102.87 53.34 0)
 			(effects
@@
 			)
 		)
-		(property "Datasheet" "~"
+		(property "Datasheet" "https://www.seielect.com/catalog/sei-rmcf_rmcp.pdf"
 			(at 100.33 129.54 0)
 			(effects
@@
 			)
 		)
-		(property "MPN" ""
+		(property "MPN" "RMCF2512FT18R0"
 			(at 100.33 129.54 0)
 			(effects
@@
 			)
 		)
-		(property "Datasheet" "~"
+		(property "Datasheet" "https://www.seielect.com/catalog/sei-rmcf_rmcp.pdf"
 			(at 100.33 160.02 0)
 			(effects
@@
 			)
 		)
-		(property "MPN" ""
+		(property "MPN" "RMCF2512FT18R0"
 			(at 100.33 160.02 0)
 			(effects
@@
 			)
 		)
-		(property "Datasheet" "~"
+		(property "Datasheet" "https://www.seielect.com/catalog/sei-rmcf_rmcp.pdf"
 			(at 100.33 83.82 0)
 			(effects
@@
 			)
 		)
-		(property "MPN" ""
+		(property "MPN" "RMCF2512FT18R0"
 			(at 100.33 83.82 0)
 			(effects
@@
 			)
 		)
-		(property "Datasheet" "~"
+		(property "Datasheet" "https://www.seielect.com/catalog/sei-rmcf_rmcp.pdf"
 			(at 100.33 144.78 0)
 			(effects
@@
 			)
 		)
-		(property "MPN" ""
+		(property "MPN" "RMCF2512FT18R0"
 			(at 100.33 144.78 0)
 			(effects
@@
 			)
 		)
-		(property "Datasheet" "~"
+		(property "Datasheet" "https://www.seielect.com/catalog/sei-rmcf_rmcp.pdf"
 			(at 100.33 175.26 0)
 			(effects
@@
 			)
 		)
-		(property "MPN" ""
+		(property "MPN" "RMCF2512FT18R0"
 			(at 100.33 175.26 0)
 			(effects
@@
 			)
 		)
-		(property "Datasheet" "~"
+		(property "Datasheet" "https://www.seielect.com/catalog/sei-rmcf_rmcp.pdf"
 			(at 100.33 68.58 0)
 			(effects
@@
 			)
 		)
-		(property "MPN" ""
+		(property "MPN" "RMCF2512FT18R0"
 			(at 100.33 68.58 0)
 			(effects
@@
 			)
 		)
-		(property "Datasheet" "~"
+		(property "Datasheet" "https://www.seielect.com/catalog/sei-rmcf_rmcp.pdf"
 			(at 100.33 114.3 0)
 			(effects
@@
 			)
 		)
-		(property "MPN" ""
+		(property "MPN" "RMCF2512FT18R0"
 			(at 100.33 114.3 0)
 			(effects
@@
 			)
 		)
-		(property "Datasheet" "~"
+		(property "Datasheet" "https://www.seielect.com/catalog/sei-rmcf_rmcp.pdf"
 			(at 100.33 190.5 0)
 			(effects
@@
 			)
 		)
-		(property "MPN" ""
+		(property "MPN" "RMCF2512FT18R0"
 			(at 100.33 190.5 0)
 			(effects
@@
 			)
 		)
-		(property "Datasheet" "~"
+		(property "Datasheet" "https://www.seielect.com/catalog/sei-rmcf_rmcp.pdf"
 			(at 100.33 205.74 0)
 			(effects
@@
 			)
 		)
-		(property "MPN" ""
+		(property "MPN" "RMCF2512FT18R0"
 			(at 100.33 205.74 0)
 			(effects

Commit message: MOre Routinggggg
Other:
- moved on the sheet: C15
Changed lines of the file:
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@@
 	(wire
 		(pts
+			(xy 114.3 44.45) (xy 114.3 43.18)
+		)
+		(stroke
+			(width 0)
+			(type default)
+		)
+	)
+	(wire
+		(pts
 			(xy 137.16 48.26) (xy 160.02 48.26)
 		)
@@
 	(wire
 		(pts
-			(xy 114.3 50.8) (xy 114.3 58.42)
+			(xy 114.3 52.07) (xy 114.3 58.42)
 		)
 		(stroke
@@
 	(symbol
 		(lib_id "Device:C")
-		(at 114.3 46.99 0)
+		(at 114.3 48.26 0)
 		(mirror y)
 		(unit 1)
@@
 		(dnp no)
 		(property "Reference" "C15"
-			(at 118.364 46.99 0)
+			(at 118.364 48.26 0)
 			(effects
 				(font
@@
 		)
 		(property "Value" "0.1uF"
-			(at 117.348 44.958 0)
+			(at 117.348 46.228 0)
 			(effects
 				(font
@@
 		)
 		(property "Footprint" "Capacitor_SMD:C_0603_1608Metric"
-			(at 113.3348 50.8 0)
+			(at 113.3348 52.07 0)
 			(effects
 				(font
@@
 		)
 		(property "Datasheet" "https://mm.digikey.com/Volume0/opasdata/d220001/medias/docus/5561/AGC%20Series.pdf"
-			(at 114.3 46.99 0)
+			(at 114.3 48.26 0)
 			(effects
 				(font
@@
 		)
 		(property "Description" "Unpolarized capacitor"
-			(at 114.3 46.99 0)
+			(at 114.3 48.26 0)
 			(effects
 				(font
@@
 		)
 		(property "MPN" "AGC0603X7R101-104KXP"
-			(at 114.3 46.99 0)
+			(at 114.3 48.26 0)
 			(effects
 				(font

Commit message: DRC error fixes
Parts:
- C15, C16, C17, C18, C19, C20, C21, C22, C23, C24, C25, C26: Digikey Part Number (none) -> 1276-6807-1-ND; MPN AGC0603X7R101-104KXP -> CL10B104KC8NNNC
- R13, R39: Digikey Part Number (none) -> RMCF0805FT100RCT-ND
- R14, R15, R16, R17, R18, R19, R20, R21, R22, R23, R24, R25, R26: Digikey Part Number (none) -> P10ADCT-ND
- R27, R28, R29, R30, R31, R32, R33, R34, R35, R36, R37, R38: Digikey Part Number (none) -> RMCF2512FT18R0CT-ND
- R40, R41, R42, R43, R44, R45, R46, R47, R48, R49, R50, R51: Digikey Part Number (none) -> 311-680GRCT-ND

Commit message: BOM updates
Parts:
- R39: Digikey Part Number RMCF0805FT100RCT-ND -> 311-100HRCT-ND; MPN ERJ-3EKF1000V -> RC0603FR-07100RL
Changed lines of the file:
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@@
 			)
 		)
-		(property "Datasheet" "https://industrial.panasonic.com/cdbs/www-data/pdf/RDA0000/AOA0000C304.pdf"
+		(property "Datasheet" "https://www.yageo.com/upload/media/product/products/datasheet/rchip/PYu-RC_Group_51_RoHS_L_12.pdf"
 			(at 81.28 34.29 0)
 			(effects
@@
 			)
 		)
-		(property "MPN" "ERJ-3EKF1000V"
+		(property "MPN" "RC0603FR-07100RL"
 			(at 81.28 34.29 0)
 			(effects
@@
 			)
 		)
-		(property "Digikey Part Number" "RMCF0805FT100RCT-ND"
+		(property "Digikey Part Number" "311-100HRCT-ND"
 			(at 81.28 34.29 0)
 			(effects
