File: BMS1/MainBMS/MainBMS.kicad_sch (KiCad schematic)
At the start: 14 parts, among them T1 Transformer_1P_1S, U1 Dev_Board_C, U2 TS2940CP33_ROG, U3 MAX33054EASA+T

Commit message: First PCB Revision
Parts:
- removed R3, R4: XX, symbol Device:R_US
- removed R5: 120, symbol Device:R_US
- removed T1: Transformer_1P_1S, symbol Device:Transformer_1P_1S
- removed U2: TS2940CP33_ROG, symbol AERO_Symbols:TS2940CP33_ROG
- removed U4: ~, symbol AERO_Symbols:LTC6820
- added J1, J2, J3: Conn_01x08, amp_seal:TE_1-776280-1_8pin_Horizontal, symbol Connector_Generic:Conn_01x08
- added U2: TS2940CP33_ROG, TS2940CP33_ROG:VREG_TS2940CP33_ROG, symbol TS2940CP33_ROG:TS2940CP33_ROG
- C1, C2: footprint (none) -> Capacitor_SMD:C_0201_0603Metric_Pad0.64x0.40mm_HandSolder
- D1: footprint (none) -> Diode_SMD:D_0201_0603Metric_Pad0.64x0.40mm_HandSolder
- D2: footprint (none) -> LED_SMD:LED_0201_0603Metric_Pad0.64x0.40mm_HandSolder
- R1, R2: footprint (none) -> Resistor_SMD:R_0201_0603Metric_Pad0.64x0.40mm_HandSolder
- U1: value Dev_Board_C -> ESP32 Dev_Board_C; footprint (none) -> AERO_Footprints:ESP32-DEV C
- U3: footprint SOIC127P600X175-8N -> AERO_Footprints:SOIC127P600X175-8N
Connections:
- net +3.3V: now also U2.3 (OUT)
- net CAN_H: now also J1.1 (Pin_1)
- net CAN_L: now also J1.4 (Pin_4)
- net GND: now also J1.3 (Pin_3), U2.2 (GND)
- net INT_12V: now also J1.2 (Pin_2), U2.1 (IN)
- net SPI1_SCK: now reaches U1.12 (MTMS/GPIO14/ADC2_CH6)
- net SPI1_SCK: now also J3.1 (Pin_1)
- net SPI1_MISO: now reaches U1.13 (*MTDI/GPIO12/ADC2_CH5)
- net SPI1_MISO: now also J3.2 (Pin_2)
- net SPI1_MOSI: now reaches U1.15 (MTCK/GPIO13/ADC2_CH4)
- net SPI1_MOSI: now also J3.3 (Pin_3)
- net SPI1_CS1: now reaches U1.23 (*MTDO/GPIO15/ADC2_CH3)
- net SPI1_CS1: now also J3.5 (Pin_5)
- net SPI0_CS1: now reaches U1.29 (*GPIO5)
- net SPI0_CS1: now also J2.1 (Pin_1)
- net SPI0_SCK: now reaches U1.30 (GPIO18)
- net SPI0_SCK: now also J2.2 (Pin_2)
- net SPI0_MISO: now reaches U1.31 (GPIO19)
- net SPI0_MISO: now also J2.3 (Pin_3)
- net SPI0_MOSI: now reaches U1.37 (GPIO23)
- net SPI0_MOSI: now also J2.5 (Pin_5)
- no-connect marks 5 -> 12
Other:
- note added: "Interface To Car"
- note added: "To BMS Section 0"
- note added: "To BMS Section 1"
- note removed: "SPI Isolation -MSTR tied VDD when on master side of interface -Slow tied to GND for clock>200kHZ"
- moved on the sheet: C2, D2, R1
